File: hardware/linetime.kicad_pcb (KiCad board)
At the start: 2 copper layers, 100 x 110 mm, 155 parts, among them IC101 STM32F7xxZxTx, IC102 ADP3335, IC103 25AA02E48, IC201 VTX-214-003-105, IC202 ADP3335, IC203 ADCMP601, IC204 ADA4528-2, IC301 ADP3335, IC302 NC7SZ04, IC303 MAX-M8Q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

Commit message: 22 airwires to go
Parts:
- removed C123: 100n, agg:0603
- removed D104: USBLC6-2P6, agg:SOT-666
- removed J101: MICROUSB, agg:MICROUSB_MOLEX_47589-0001
- removed P102: SWD_TC, agg:TC2030-NL
- removed R109: 10k, agg:0603
- added R1: 10k, agg:0603, F.Cu at (61.9, 101.7)
- added R2: 10k, agg:0603, F.Cu at (58.7, 101.7)
- added R?: 22, agg:0603, F.Cu at (55.6, 84.5)
- C401: footprint agg:0805 -> agg:1206
- U101: moved to B.Cu
- moved IC101 100.0 mm to (71.5, 124.8), turned to 90 degrees
- moved C117 94.7 mm to (85.5, 114.6), turned to 90 degrees
- moved C106 92.1 mm to (75.0, 111.1), turned to 90 degrees
- moved C115 89.7 mm to (85.9, 121.2)
- moved U101 88.9 mm to (59.6, 145.3), turned to 0 degrees
- moved C111 88.2 mm to (69.5, 111.1), turned to 90 degrees
- moved R403 83.0 mm to (80.8, 71.9), turned to 90 degrees
- moved C108 78.7 mm to (78.2, 138.8), turned to 270 degrees
- moved C118 77.9 mm to (61.4, 110.8), turned to 180 degrees
- moved R102 77.9 mm to (56.8, 130.0), turned to 180 degrees
- moved C110 77.2 mm to (61.4, 112.3), turned to 180 degrees
- moved C102 77.1 mm to (84.0, 114.6), turned to 90 degrees
- moved C103 75.0 mm to (86.2, 134.1), turned to 270 degrees
- moved D103 73.3 mm to (53.7, 131.5)
- moved C116 72.6 mm to (56.8, 133.2), turned to 180 degrees
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Connections:
- IC101 pad 10: /~CE -> Net-(IC101-Pad10)
- IC101 pad 100: Net-(IC101-Pad100) -> /SD2100_SCL
- IC101 pad 11: /~PGOOD -> Net-(IC101-Pad11)
- IC101 pad 12: /~CHG -> Net-(IC101-Pad12)
- IC101 pad 135: Net-(IC101-Pad135) -> /LED1
- IC101 pad 136: Net-(IC101-Pad136) -> /LED2
- IC101 pad 137: Net-(IC101-Pad137) -> /LED3
- IC101 pad 54: /SD2100_SCL -> Net-(IC101-Pad54)
- IC101 pad 55: /CS2100_SDA -> Net-(IC101-Pad55)
- IC101 pad 73: Net-(IC101-Pad73) -> /~CHG
- IC101 pad 74: /VUSB -> /~PGOOD
- IC101 pad 75: /USB_D- -> /~CE
- IC101 pad 76: /USB_D+ -> Net-(IC101-Pad76)
- IC101 pad 87: /LED1 -> Net-(IC101-Pad87)
- IC101 pad 88: /LED2 -> Net-(IC101-Pad88)
- IC101 pad 89: /LED3 -> Net-(IC101-Pad89)
- IC101 pad 99: Net-(IC101-Pad99) -> /CS2100_SDA
- IC304 pad 3: /CS2100_CLK -> Net-(IC304-Pad3)
Routing:
- net 3v3: track 22.9 -> 514.0 mm, vias 0 -> 10
- net GND: track 57.1 -> 456.8 mm, vias 23 -> 144
- net /TOUCH_~CS: track 0.00 -> 96.4 mm, vias 0 -> 4
- net VCC: track 32.8 -> 129.0 mm, vias 2 -> 3
- net /TOUCH_INT: track 0.00 -> 90.2 mm, vias 0 -> 4
- net /ROM_SI: track 0.00 -> 86.1 mm
- net /ROM_SO: track 0.00 -> 84.2 mm, vias 0 -> 2
- net /ROM_SCK: track 0.00 -> 78.6 mm, vias 0 -> 2
- net /BACKLIGHT: track 0.00 -> 72.2 mm, vias 0 -> 6
- net /CS2100_CLK: track 0.00 -> 67.0 mm, vias 0 -> 4
- net Net-(IC402-Pad15): track 0.00 -> 64.5 mm, vias 0 -> 2
- net /GPS_~RESET: track 0.00 -> 64.4 mm
- net /linetime_ui/Y-: track 0.00 -> 62.4 mm, vias 0 -> 4
- net /uSD_DAT0: track 0.00 -> 61.3 mm, vias 0 -> 4
- net /MDIO: track 0.00 -> 60.9 mm, vias 0 -> 4
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- added copper zone on F.Cu, net GND
Other:
- board size 100 x 110 mm -> 100 x 100 mm

Commit message: 17 airwires
Parts:
- moved C112 1.87 mm to (87.7, 125.6)
Routing:
- net /HSYNC: track 0.00 -> 78.9 mm, vias 0 -> 7
- net /R7: track 0.00 -> 49.5 mm, vias 0 -> 5
- net /VSYNC: track 0.00 -> 49.1 mm, vias 0 -> 3
- net /DOTCLK: track 0.00 -> 48.8 mm, vias 0 -> 5
- net /DE: track 0.00 -> 47.9 mm, vias 0 -> 5
- net GND: track 456.8 -> 489.3 mm, vias 144 -> 146
- net /R6: track 0.00 -> 12.4 mm, vias 0 -> 1
- net /V_BATT_MON: track 90.0 -> 96.5 mm
- net /I_CHG: track 104.6 -> 110.8 mm
- net Net-(IC402-Pad15): track 64.5 -> 60.0 mm, vias 2 -> 4
- net 3v3: track 514.0 -> 517.7 mm
- net /MAINS_ZC: track 78.2 -> 81.5 mm
- net Net-(D602-Pad2): track 5.97 -> 4.16 mm
- net /SOUNDER_~SD: track 36.1 -> 37.4 mm

Commit message: 4 to go!!
Routing:
- net /R4: track 0.00 -> 102.3 mm, vias 0 -> 11
- net /R5: track 0.00 -> 100.8 mm, vias 0 -> 11
- net /G6: track 0.00 -> 75.9 mm, vias 0 -> 7
- net /B6: track 0.00 -> 67.0 mm, vias 0 -> 1
- net /B7: track 0.00 -> 66.1 mm, vias 0 -> 1
- net /G7: track 0.00 -> 64.2 mm, vias 0 -> 9
- net /G5: track 0.00 -> 48.5 mm, vias 0 -> 5
- net /G4: track 0.00 -> 46.7 mm, vias 0 -> 5
- net /R3: track 0.00 -> 44.6 mm, vias 0 -> 5
- net /B4: track 0.00 -> 43.2 mm, vias 0 -> 7
- net /G3: track 0.00 -> 41.9 mm, vias 0 -> 5
- net /B5: track 0.00 -> 36.7 mm, vias 0 -> 5
- net /R6: track 12.4 -> 45.6 mm, vias 1 -> 5
- net GND: track 489.3 -> 498.3 mm, vias 146 -> 148
- net /BACKLIGHT: track 72.2 -> 77.2 mm
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
Commit message: 565RGB and 2 airwires left yay
Parts:
- moved C117 1.70 mm to (84.8, 116.2), turned to 0 degrees
- moved C102 0.80 mm to (84.8, 114.7), turned to 0 degrees
Routing:
- net /B3: track 0.00 -> 67.1 mm, vias 0 -> 9
- net /G2: track 0.00 -> 31.1 mm, vias 0 -> 3
- net /BACKLIGHT: track 77.2 -> 80.4 mm
- net /R6: track 45.6 -> 48.3 mm
- net 3v3: track 522.0 -> 524.6 mm
- net Net-(C117-Pad1): track 4.13 -> 1.89 mm
- net GND: track 498.3 -> 500.3 mm
- net /~CHG: track 81.8 -> 80.6 mm
- net /~PGOOD: track 81.1 -> 79.9 mm
- net /~CE: track 79.5 -> 78.4 mm
- net /B6: track 67.0 -> 66.0 mm
- net /B7: track 66.1 -> 65.2 mm
- net /B5: track 36.7 -> 35.9 mm
- net /G6: track 75.9 -> 75.1 mm

Commit message: cleaned up all the fast lines
Parts:
- removed C412: 10µ, agg:0603
- removed D401: 1N4148, agg:SOD-323
- removed L202: ~, agg:0603
- removed R?: 22, agg:0603
- added R206: 100, agg:0603, F.Cu at (116.1, 119.1)
- added R303: 33, agg:0603, F.Cu at (55.6, 84.5)
- added R411: 33, agg:0603, F.Cu at (57.7, 124.1)
- added R412: 33, agg:0603, F.Cu at (54.7, 124.1)
- added R413: 33, agg:0603, F.Cu at (56.2, 124.1)
- C207: value ~ -> 1n
- R205: value 22 -> 33
- moved R408 47.5 mm to (77.0, 90.6), turned to 270 degrees
- moved R405 42.2 mm to (75.5, 90.6), turned to 270 degrees
- moved R407 41.2 mm to (74.0, 90.6), turned to 270 degrees
- moved R404 40.2 mm to (72.5, 90.6), turned to 270 degrees
- moved C406 6.86 mm to (79.3, 89.8), turned to 180 degrees
- moved C407 6.14 mm to (79.3, 88.3), turned to 180 degrees
- moved R1 3.83 mm to (58.1, 102.2), turned to 270 degrees
- moved R410 3.57 mm to (79.0, 94.5)
- moved C207 2.53 mm to (116.9, 116.7), turned to 0 degrees
- moved R2 2.15 mm to (56.6, 102.2), turned to 270 degrees
- moved C114 1.05 mm to (57.9, 121.7)
- moved R409 0.90 mm to (69.9, 93.9), turned to 90 degrees
- moved C106 0.81 mm to (74.2, 111.0)
- moved C113 0.35 mm to (56.8, 126.8)
Connections:
- IC101 pad 76: Net-(IC101-Pad76) -> /PHY_~RST
- IC402 pad 19: /TXEN -> Net-(IC402-Pad19)
- IC402 pad 20: /TXD0 -> Net-(IC402-Pad20)
- IC402 pad 21: /TXD1 -> Net-(IC402-Pad21)
- IC402 pad 24: Net-(C412-Pad1) -> /PHY_~RST
- R201 pad 2: Net-(L202-Pad2) -> Net-(C207-Pad1)
- R410 pad 1: 3v3 -> /PHY_~RST
- R410 pad 2: Net-(C412-Pad1) -> GND
- T201 pad 8: Net-(C207-Pad1) -> Net-(R206-Pad2)
Routing:
- net Net-(IC402-Pad15): track 60.0 -> 3.24 mm, vias 4 -> 0
- net Net-(IC402-Pad12): track 60.0 -> 3.27 mm, vias 4 -> 0
- net Net-(IC402-Pad21): track 0.00 -> 56.3 mm, vias 0 -> 2
- net Net-(IC402-Pad13): track 59.3 -> 3.05 mm, vias 4 -> 0
- net Net-(IC402-Pad20): track 0.00 -> 55.0 mm, vias 0 -> 2
- net Net-(IC402-Pad19): track 0.00 -> 54.6 mm, vias 0 -> 2
- net Net-(IC402-Pad16): track 56.1 -> 4.23 mm, vias 2 -> 0
- net /TXD1: track 57.4 -> 6.99 mm, vias 2 -> 0
- net /TXD0: track 54.8 -> 5.43 mm, vias 2 -> 0
- net /TXEN: track 52.1 -> 3.27 mm, vias 2 -> 0
- net /REF_CLK: track 2.64 -> 46.0 mm, vias 0 -> 2
- net /RXD0: track 2.90 -> 45.5 mm, vias 0 -> 2
- net /RXD1: track 3.33 -> 45.1 mm, vias 0 -> 2
- net /CRS_DV: track 3.33 -> 45.0 mm, vias 0 -> 2
- net /PHY_~RST: track 0.00 -> 39.5 mm, vias 0 -> 2
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
Commit message: goodness. routed all airwires.
Routing:
- net /R2: track 0.00 -> 101.3 mm, vias 0 -> 9
- net /B2: track 0.00 -> 74.6 mm, vias 0 -> 3
- net /B6: track 63.4 -> 60.0 mm
- net /B7: track 62.7 -> 59.4 mm
- net /R6: track 48.2 -> 45.0 mm
- net /R4: track 102.5 -> 100.9 mm
- net /R5: track 97.7 -> 96.7 mm
- net /G5: track 48.6 -> 47.7 mm
- net /CS2100_CLK: track 65.2 -> 64.4 mm
- net /uSD_CMD: track 43.2 -> 43.8 mm
- net /DE: track 47.6 -> 47.0 mm
- net /GPS_TXD: track 62.9 -> 62.3 mm
- net GND: track 500.2 -> 500.7 mm
- net 3v3: track 520.8 -> 521.1 mm, vias 16 -> 18

Commit message: tidying
Routing:
- net GND: track 500.7 -> 519.6 mm, vias 147 -> 149
- net 3v3: track 521.1 -> 511.2 mm
- net /R4: track 100.9 -> 96.7 mm
- net /B3: track 68.3 -> 64.3 mm
- net /nRST: track 43.3 -> 40.4 mm, vias 5 -> 3
- net /MAINS_ZC: track 76.5 -> 78.9 mm
- net /HSYNC: track 78.1 -> 75.8 mm
- net /G6: track 74.6 -> 73.0 mm
- net /CS2100_CLK: track 64.4 -> 63.1 mm
- net /R3: track 39.7 -> 40.9 mm
- net /uSD_DAT0: track 54.0 -> 55.2 mm, vias 2 -> 4
- net /R2: track 101.3 -> 102.3 mm
- net /BACKLIGHT: track 79.2 -> 78.2 mm
- net /MDIO: track 60.1 -> 59.2 mm
- net /MDC: track 53.7 -> 52.9 mm
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Other:
- board text added: "2016-12-19"
- board text added: "LINETIME r1 ADAM GREIG"
- board text added: "WARNING HIGH VOLTAGE"

Commit message: gerbers to manufacturing. gulp.
Routing:
- net GND: track 519.6 -> 564.8 mm, vias 149 -> 159
- net /uSD_CMD: track 43.8 -> 41.9 mm
