File: hardware/linetime.sch (KiCad schematic (older format))
At the start: 3 parts

Commit message: schematic basically done...
Parts:
- added C101, C102, C105, C106, C107, C108, C109, C110, C111, C112, C113, C114, C115, C116, C119, C123: 100n, agg:0603, symbol C
- added C103: 4µ7, agg:0603, symbol C
- added C104, C120, C122: 1µ, agg:0603, symbol C
- added C117, C118: 2µ2, agg:0603, symbol C
- added C121: 10n, agg:0603, symbol C
- added D101, D102, D103: LED, agg:0603-LED, symbol LED
- added D104: USBLC6-2P6, agg:SOT-666, symbol USBLC6-2P6
- added IC101: STM32F7xxZxTx, agg:LQFP-144, symbol STM32F7xxZxTx
- added IC102: ADP3335, agg:MSOP-8, symbol ADP3335
- added J101: MICROUSB, agg:MICROUSB_MOLEX_47589-0001, symbol MICROUSB
- added R101, R102, R103: 1k, agg:0603, symbol R
- added R104, R105, R106, R107, R108: 47k, agg:0603, symbol R
- added R109: 10k, agg:0603, symbol R
- added U101: MICROSD, agg:MICROSD_MOLEX_503398-1892, symbol MICROSD
- gave numbers to parts that had none: 3
Connections:
- net ROM_SCK: now reaches IC103.1 (SCK)
- net ROM_SCK: now also IC101.19 (PF7)
- net GND: now reaches IC103.2 (VSS)
- net GND: now also P101.3 (GND), P101.5 (GND), P101.9 (GND), P102.5 (GND), C101.2, C102.2, C103.2, C104.2, C105.2, C106.2, C107.2, C108.2, C109.2, C110.2, C111.2, C112.2, C113.2, C114.2, C115.2, C116.2, C117.2, C118.2, C119.2, C120.2, C122.2, C123.2, D101.1, D102.1, D103.1, D104.2 (GND), IC101.107 (VSS), IC101.120 (VSS), IC101.130 (VSS), IC101.138 (BOOT0), IC101.16 (VSS), IC101.31 (VSSA), IC101.38 (VSS), IC101.51 (VSS), IC101.61 (VSS), IC101.83 (VSS), IC101.94 (VSS), IC102.4 (GND), J101.5 (GND), U101.6 (VSS), U101.9 (SHIELD)
- net ROM_SI: now reaches IC103.3 (SI)
- net ROM_SI: now also IC101.21 (PF9)
- net ROM_SO: now reaches IC103.4 (SO)
- net ROM_SO: now also IC101.20 (PF8)
- net ROM_~CS: now reaches IC103.5 (~CS)
- net ROM_~CS: now also IC101.22 (PF10)
- net 3v3: now reaches IC103.6 (VDD)
- net 3v3: now also P101.1 (VTref), P102.1 (VDD), C101.1, C102.1, C103.1, C104.1, C105.1, C106.1, C107.1, C108.1, C109.1, C110.1, C111.1, C112.1, C113.1, C114.1, C115.1, C116.1, C119.1, C121.2, C122.1, C123.1, IC101.108 (VDD), IC101.121 (VDDSDMMC), IC101.131 (VDD), IC101.143 (PDR_ON), IC101.144 (VDD), IC101.17 (VDD), IC101.30 (VDD), IC101.32 (VREF+), IC101.33 (VDDA), IC101.39 (VDD), IC101.52 (VDD), IC101.6 (VBAT), IC101.62 (VDD), IC101.72 (VDD), IC101.84 (VDD), IC101.95 (VDDUSB), IC102.1 (OUT), IC102.2 (OUT), IC102.3 (OUT), R104.1, R105.1, R106.1, R107.1, R108.1, U101.4 (VDD)
- net nRST: now reaches P101.10 (nRESET)
- net nRST: now also P102.3 (~RST), IC101.25 (NRST)
- net SWDIO: now reaches P101.2 (SWDIO/TMS)
- net SWDIO: now also P102.2 (SWDIO), IC101.105 (PA13)
- net SWCLK: now reaches P101.4 (SWDCLK/TCK)
- net SWCLK: now also P102.4 (SWDCLK), IC101.109 (PA14)
- new net: D104.5 (VBUS), J101.1 (VCC), R109.1
- new net: D104.6 (I/O1), J101.2 (D-)
- new net: D104.4 (I/O2), J101.3 (D+)
- new net: R105.2, U101.1 (DAT2)
- new net: R108.2, U101.2 (DAT3)
- new net: R107.2, U101.8 (DAT1)
- new net: C121.1, IC102.5 (NR)
- new net: C118.1, IC101.106 (VCAP2)
- new net: C117.1, IC101.71 (VCAP1)
- new net: D101.2, R101.2
- new net: D102.2, R102.2
- new net: D103.2, R103.2
- new net B2: IC101.125 (PG10)
- new net B3: IC101.79 (PD10)
- new net B4: IC101.65 (PE12)
- new net B5: IC101.37 (PA3)
- new net B6: IC101.139 (PB8)
- new net B7: IC101.140 (PB9)
- new net BACKLIGHT: IC101.81 (PD12)
- new net CRS_DV: IC101.43 (PA7)
- new net CS2100_CLK: IC101.23 (PH0)
- new net CS2100_SDA: IC101.55 (PF15)
- new net DE: IC101.66 (PE13)
- new net DOTCLK: IC101.67 (PE14)
- new net G2: IC101.42 (PA6)
- new net G3: IC101.64 (PE11)
- new net G4: IC101.69 (PB10)
- new net G5: IC101.70 (PB11)
- new net G6: IC101.97 (PC7)
- new net G7: IC101.93 (PG8)
- new net GPS_PPS: IC101.133 (PB3)
- new net GPS_RXD: IC101.119 (PD5)
- new net GPS_TXD: IC101.122 (PD6)
- new net GPS_~RESET: IC101.118 (PD4)
- new net HSYNC: IC101.96 (PC6)
- new net I_CHG: IC101.13 (PF3)
- new net LED1: IC101.87 (PG2), R101.1
- new net LED2: IC101.88 (PG3), R102.1
- new net LED3: IC101.89 (PG4), R103.1
- new net MAINS_BIAS: IC101.29 (PC3)
- new net MAINS_WAVE: IC101.28 (PC2)
- new net MAINS_ZC: IC101.110 (PA15)
- new net MDC: IC101.27 (PC1)
- new net MDIO: IC101.36 (PA2)
- new net R2: IC101.111 (PC10)
- new net R3: IC101.46 (PB0)
- new net R4: IC101.103 (PA11)
- new net R5: IC101.104 (PA12)
- new net R6: IC101.47 (PB1)
- new net R7: IC101.68 (PE15)
- new net REF_CLK: IC101.35 (PA1)
- new net RXD0: IC101.44 (PC4)
- new net RXD1: IC101.45 (PC5)
- new net SD2100_SCL: IC101.54 (PF14)
- new net SOUNDER: IC101.41 (PA5)
- new net SOUNDER_~SD: IC101.48 (PB2)
- new net TFT_DCX: IC101.2 (PE3)
- new net TFT_RESET: IC101.4 (PE5)
- new net TFT_SCL: IC101.1 (PE2)
- new net TFT_SDA: IC101.5 (PE6)
- new net TFT_~CS: IC101.3 (PE4)
- new net TOUCH_INT: IC101.15 (PF5)
- new net TOUCH_~CS: IC101.18 (PF6)
- new net TXD0: IC101.128 (PG13)
- new net TXD1: IC101.129 (PG14)
- new net TXEN: IC101.126 (PG11)
- new net USB_D+: D104.3 (I/O2), IC101.76 (PB15)
- new net USB_D-: D104.1 (I/O1), IC101.75 (PB14)
- new net VCC: C120.1, IC102.6 (SD), IC102.7 (IN), IC102.8 (IN)
- new net VSYNC: IC101.40 (PA4)
- new net VUSB: IC101.74 (PB13), R109.2
- new net V_BATT/2: IC101.14 (PF4)
- new net uSD_CLK: IC101.113 (PC12), U101.5 (CLK)
- new net uSD_CMD: IC101.116 (PD2), R106.2, U101.3 (CMD)
- new net uSD_DAT0: IC101.98 (PC8), R104.2, U101.7 (DAT0)
- new net ~CE: IC101.10 (PF0)
- new net ~CHG: IC101.12 (PF2)
- new net ~PGOOD: IC101.11 (PF1)
- no-connect marks 0 -> 50
Other:
- note added: "3v3 LDO for digital supply"
- note added: "Debug/programming Interface"
- note added: "Indicator LEDs"
- note added: "MicroSD Holder"
- note added: "ROM with MAC address"
- note added: "USB Connector"
- note added: "VBAT"
- note added: "VDD"
- note added: "VDD@108"
- note added: "VDD@131"
- note added: "VDD@144"
- note added: "VDD@17"
- note added: "VDD@30"
- note added: "VDD@39"
- note added: "VDD@52"
- note added: "VDD@62"
- note added: "VDD@72"
- note added: "VDD@84"
- note added: "VDDA & VREF+"
- note added: "VDDSDMMC"
- note added: "VDDUSB"
- moved on the sheet: IC103, P101, P102

Commit message: WIP routing
Connections:
- net USB_D+: now also D104.1 (I/O1); no longer D104.3 (I/O2)
- net USB_D-: now also D104.3 (I/O2); no longer D104.1 (I/O1)
- net at J101.2 (D-): now also D104.4 (I/O2); no longer D104.6 (I/O1)
- net at J101.3 (D+): now also D104.6 (I/O1); no longer D104.4 (I/O2)
- net V_BATT/2 renamed V_BATT_MON
Changed lines of the file:
@@
 F6 "~CHG" O L 14850 2050 40
 F7 "I_CHG" O L 14850 2150 40
-F8 "V_BATT/2" O L 14850 2250 40
+F8 "V_BATT_MON" O L 14850 2250 40
 $EndSheet
 $Sheet
@@
 $EndComp
 $Comp
-L VCC #PWR01
+L VCC #PWR130
 U 1 1 584C7DBB
 P 14500 1700
-F 0 "#PWR01" H 14500 1810 50  0001 L CNN
+F 0 "#PWR130" H 14500 1810 50  0001 L CNN
 F 1 "VCC" H 14500 1790 50  0000 C CNN
 F 2 "" H 14500 1700 60  0001 C CNN
@@
 $EndComp
 $Comp
-L GND #PWR02
+L GND #PWR135
 U 1 1 584C9ADD
 P 15700 8500
-F 0 "#PWR02" H 15570 8540 50  0001 L CNN
+F 0 "#PWR135" H 15570 8540 50  0001 L CNN
 F 1 "GND" H 15700 8400 50  0000 C CNN
 F 2 "" H 15700 8500 60  0001 C CNN
@@
 $EndComp
 $Comp
-L GND #PWR03
+L GND #PWR131
 U 1 1 584C9AED
 P 14700 8650
-F 0 "#PWR03" H 14570 8690 50  0001 L CNN
+F 0 "#PWR131" H 14570 8690 50  0001 L CNN
 F 1 "GND" H 14700 8550 50  0000 C CNN
 F 2 "" H 14700 8650 60  0001 C CNN
@@
 3v3 LDO for digital supply
 $Comp
-L VCC #PWR04
+L VCC #PWR129
 U 1 1 584C9B0C
 P 14450 8250
-F 0 "#PWR04" H 14450 8360 50  0001 L CNN
+F 0 "#PWR129" H 14450 8360 50  0001 L CNN
 F 1 "VCC" H 14450 8340 50  0000 C CNN
 F 2 "" H 14450 8250 60  0001 C CNN
@@
 $EndComp
 $Comp
-L 3v3 #PWR05
+L 3v3 #PWR136
 U 1 1 584C9D95
 P 15800 8250
-F 0 "#PWR05" H 15800 8360 50  0001 L CNN
+F 0 "#PWR136" H 15800 8360 50  0001 L CNN
 F 1 "3v3" H 15800 8340 50  0000 C CNN
 F 2 "" H 15800 8250 60  0001 C CNN
@@
 SD2100_SCL
 Text Label 14750 2250 2    40   ~ 0
-V_BATT/2
+V_BATT_MON
 Text Label 14750 2150 2    40   ~ 0
 I_CHG
@@
 MAINS_ZC
 $Comp
-L GND #PWR06
+L GND #PWR134
 U 1 1 584D3535
 P 15600 9350
-F 0 "#PWR06" H 15470 9390 50  0001 L CNN
+F 0 "#PWR134" H 15470 9390 50  0001 L CNN
 F 1 "GND" H 15600 9250 50  0000 C CNN
 F 2 "" H 15600 9350 60  0001 C CNN
@@
 $EndComp
 $Comp
-L GND #PWR07
+L GND #PWR138
 U 1 1 584D39B1
 P 15800 9350
-F 0 "#PWR07" H 15670 9390 50  0001 L CNN
+F 0 "#PWR138" H 15670 9390 50  0001 L CNN
 F 1 "GND" H 15800 9250 50  0000 C CNN
 F 2 "" H 15800 9350 60  0001 C CNN
@@
 NoConn ~ 15450 7700
 $Comp
-L GND #PWR08
+L GND #PWR132
 U 1 1 584D6796
 P 15350 7850
-F 0 "#PWR08" H 15220 7890 50  0001 L CNN
+F 0 "#PWR132" H 15220 7890 50  0001 L CNN
 F 1 "GND" H 15350 7750 50  0000 C CNN
 F 2 "" H 15350 7850 60  0001 C CNN
@@
 USB Connector
 $Comp
-L 3v3 #PWR09
+L 3v3 #PWR124
 U 1 1 584DBAF6
 P 12750 7300
-F 0 "#PWR09" H 12750 7410 50  0001 L CNN
+F 0 "#PWR124" H 12750 7410 50  0001 L CNN
 F 1 "3v3" H 12750 7390 50  0000 C CNN
 F 2 "" H 12750 7300 60  0001 C CNN
@@
 $EndComp
 $Comp
-L GND #PWR010
+L GND #PWR121
 U 1 1 584DBE42
 P 12550 7450
-F 0 "#PWR010" H 12420 7490 50  0001 L CNN
+F 0 "#PWR121" H 12420 7490 50  0001 L CNN
 F 1 "GND" H 12550 7350 50  0000 C CNN
 F 2 "" H 12550 7450 60  0001 C CNN
@@
 $EndComp
 $Comp
-L GND #PWR011
+L GND #PWR125
 U 1 1 584DC198
 P 13750 7400
-F 0 "#PWR011" H 13620 7440 50  0001 L CNN
+F 0 "#PWR125" H 13620 7440 50  0001 L CNN
 F 1 "GND" H 13750 7300 50  0000 C CNN
 F 2 "" H 13750 7400 60  0001 C CNN
@@
 $EndComp
 $Comp
-L 3v3 #PWR012
+L 3v3 #PWR118
 U 1 1 584E1F30
 P 12200 7450
-F 0 "#PWR012" H 12200 7560 50  0001 L CNN
+F 0 "#PWR118" H 12200 7560 50  0001 L CNN
 F 1 "3v3" H 12200 7540 50  0000 C CNN
 F 2 "" H 12200 7450 60  0001 C CNN
@@
 $EndComp
 $Comp
-L GND #PWR013
+L GND #PWR127
 U 1 1 584B90B9
 P 13850 7900
-F 0 "#PWR013" H 13720 7940 50  0001 L CNN
+F 0 "#PWR127" H 13720 7940 50  0001 L CNN
 F 1 "GND" H 13850 7800 50  0000 C CNN
 F 2 "" H 13850 7900 60  0001 C CNN
@@
 $EndComp
 $Comp
-L 3v3 #PWR014
+L 3v3 #PWR119
 U 1 1 584BAEC8
 P 12500 8500
-F 0 "#PWR014" H 12500 8610 50  0001 L CNN
+F 0 "#PWR119" H 12500 8610 50  0001 L CNN
 F 1 "3v3" H 12500 8590 50  0000 C CNN
 F 2 "" H 12500 8500 60  0001 C CNN
@@
 $EndComp
 $Comp
-L GND #PWR015
+L GND #PWR120
 U 1 1 584BB271
 P 12500 9000
-F 0 "#PWR015" H 12370 9040 50  0001 L CNN
+F 0 "#PWR120" H 12370 9040 50  0001 L CNN
 F 1 "GND" H 12500 8900 50  0000 C CNN
 F 2 "" H 12500 9000 60  0001 C CNN
@@
 nRST
 $Comp
-L 3v3 #PWR016
+L 3v3 #PWR122
 U 1 1 584BC2E0
 P 12600 9300
-F 0 "#PWR016" H 12600 9410 50  0001 L CNN
+F 0 "#PWR122" H 12600 9410 50  0001 L CNN
 F 1 "3v3" H 12600 9390 50  0000 C CNN
 F 2 "" H 12600 9300 60  0001 C CNN
@@
 $EndComp
 $Comp
-L GND #PWR017
+L GND #PWR123
 U 1 1 584BC563
 P 12600 9600
-F 0 "#PWR017" H 12470 9640 50  0001 L CNN
+F 0 "#PWR123" H 12470 9640 50  0001 L CNN
 F 1 "GND" H 12600 9500 50  0000 C CNN
 F 2 "" H 12600 9600 60  0001 C CNN
@@
 F 4 "1295310" H 14550 7050 50  0001 L CNN "Farnell"
 	1    14850 7550
-	1    0    0    -1
-$EndComp
-$Comp
-L GND #PWR018
+	1    0    0    1
+$EndComp
+$Comp
+L GND #PWR128
 U 1 1 584C2515
 P 14300 7550
-F 0 "#PWR018" H 14170 7590 50  0001 L CNN
+F 0 "#PWR128" H 14170 7590 50  0001 L CNN
 F 1 "GND" H 14300 7450 50  0000 C CNN
 F 2 "" H 14300 7550 60  0001 C CNN
@@
 $EndComp
 $Comp
-L 3v3 #PWR019
+L 3v3 #PWR113
 U 1 1 5850C0F5
 P 2650 1500
-F 0 "#PWR019" H 2650 1610 50  0001 L CNN
+F 0 "#PWR113" H 2650 1610 50  0001 L CNN
 F 1 "3v3" H 2650 1590 50  0000 C CNN
 F 2 "" H 2650 1500 60  0001 C CNN
@@
 $EndComp
 $Comp
-L GND #PWR020
+L GND #PWR114
 U 1 1 5850DD9F
 P 2650 4400
-F 0 "#PWR020" H 2520 4440 50  0001 L CNN
+F 0 "#PWR114" H 2520 4440 50  0001 L CNN
 F 1 "GND" H 2650 4300 50  0000 C CNN
 F 2 "" H 2650 4400 60  0001 C CNN
@@
 SOUNDER
 $Comp
-L 3v3 #PWR021
+L 3v3 #PWR133
 U 1 1 58536723
 P 15600 9150
-F 0 "#PWR021" H 15600 9260 50  0001 L CNN
+F 0 "#PWR133" H 15600 9260 50  0001 L CNN
 F 1 "3v3" H 15600 9240 50  0000 C CNN
 F 2 "" H 15600 9150 60  0001 C CNN
@@
 $EndComp
 $Comp
-L 3v3 #PWR022
+L 3v3 #PWR137
 U 1 1 58536C0A
 P 15800 9150
-F 0 "#PWR022" H 15800 9260 50  0001 L CNN
+F 0 "#PWR137" H 15800 9260 50  0001 L CNN
 F 1 "3v3" H 15800 9240 50  0000 C CNN
 F 2 "" H 15800 9150 60  0001 C CNN
@@
 $EndComp
 $Comp
-L 3v3 #PWR023
+L 3v3 #PWR126
 U 1 1 5853786D
 P 13850 7700
-F 0 "#PWR023" H 13850 7810 50  0001 L CNN
+F 0 "#PWR126" H 13850 7810 50  0001 L CNN
 F 1 "3v3" H 13850 7790 50  0000 C CNN
 F 2 "" H 13850 7700 60  0001 C CNN
@@
 MAINS_ZC
 Text Label 4250 7050 0    40   ~ 0
-V_BATT/2
+V_BATT_MON
 Text Label 4250 6950 0    40   ~ 0
 I_CHG
@@
 $EndComp
 $Comp
-L GND #PWR024
+L GND #PWR111
 U 1 1 58597AB1
 P 2450 3450
-F 0 "#PWR024" H 2320 3490 50  0001 L CNN
+F 0 "#PWR111" H 2320 3490 50  0001 L CNN
 F 1 "GND" H 2450 3350 50  0000 C CNN
 F 2 "" H 2450 3450 60  0001 C CNN
@@
 $EndComp
 $Comp
-L GND #PWR025
+L GND #PWR109
 U 1 1 58597EDC
 P 2250 3450
-F 0 "#PWR025" H 2120 3490 50  0001 L CNN
+F 0 "#PWR109" H 2120 3490 50  0001 L CNN
 F 1 "GND" H 2250 3350 50  0000 C CNN
 F 2 "" H 2250 3450 60  0001 C CNN
@@
 $EndComp
 $Comp
-L 3v3 #PWR026
+L 3v3 #PWR101
 U 1 1 5859F241
 P 1000 1100
-F 0 "#PWR026" H 1000 1210 50  0001 L CNN
+F 0 "#PWR101" H 1000 1210 50  0001 L CNN
 F 1 "3v3" H 1000 1190 50  0000 C CNN
 F 2 "" H 1000 1100 60  0001 C CNN
@@
 $EndComp
 $Comp
-L 3v3 #PWR027
+L 3v3 #PWR102
 U 1 1 585A01BC
 P 1000 1600
-F 0 "#PWR027" H 1000 1710 50  0001 L CNN
+F 0 "#PWR102" H 1000 1710 50  0001 L CNN
 F 1 "3v3" H 1000 1690 50  0000 C CNN
 F 2 "" H 1000 1600 60  0001 C CNN
@@
 $EndComp
 $Comp
-L 3v3 #PWR028
+L 3v3 #PWR103
 U 1 1 585A0D13
 P 1000 2100
-F 0 "#PWR028" H 1000 2210 50  0001 L CNN
+F 0 "#PWR103" H 1000 2210 50  0001 L CNN
 F 1 "3v3" H 1000 2190 50  0000 C CNN
 F 2 "" H 1000 2100 60  0001 C CNN
@@
 $EndComp
 $Comp
-L GND #PWR029
+L GND #PWR108
 U 1 1 585A1B30
 P 2250 1900
-F 0 "#PWR029" H 2120 1940 50  0001 L CNN
+F 0 "#PWR108" H 2120 1940 50  0001 L CNN
 F 1 "GND" H 2250 1800 50  0000 C CNN
 F 2 "" H 2250 1900 60  0001 C CNN
@@
 $EndComp
 $Comp
-L GND #PWR030
+L GND #PWR107
 U 1 1 585A2B46
 P 2250 1400
-F 0 "#PWR030" H 2120 1440 50  0001 L CNN
+F 0 "#PWR107" H 2120 1440 50  0001 L CNN
 F 1 "GND" H 2250 1300 50  0000 C CNN
 F 2 "" H 2250 1400 60  0001 C CNN
@@
 $EndComp
 $Comp
-L GND #PWR031
+L GND #PWR106
 U 1 1 585A3B41
 P 2000 2400
-F 0 "#PWR031" H 1870 2440 50  0001 L CNN
+F 0 "#PWR106" H 1870 2440 50  0001 L CNN
 F 1 "GND" H 2000 2300 50  0000 C CNN
 F 2 "" H 2000 2400 60  0001 C CNN
@@
 $EndComp
 $Comp
-L 3v3 #PWR032
+L 3v3 #PWR104
 U 1 1 585A5365
 P 1000 2600
-F 0 "#PWR032" H 1000 2710 50  0001 L CNN
+F 0 "#PWR104" H 1000 2710 50  0001 L CNN
 F 1 "3v3" H 1000 2690 50  0000 C CNN
 F 2 "" H 1000 2600 60  0001 C CNN
@@
 $EndComp
 $Comp
-L GND #PWR033
+L GND #PWR105
 U 1 1 585A5B63
 P 1500 2900
-F 0 "#PWR033" H 1370 2940 50  0001 L CNN
+F 0 "#PWR105" H 1370 2940 50  0001 L CNN
 F 1 "GND" H 1500 2800 50  0000 C CNN
 F 2 "" H 1500 2900 60  0001 C CNN
@@
 VDD@144
 $Comp
-L 3v3 #PWR034
+L 3v3 #PWR112
 U 1 1 585BA0D6
 P 2500 4550
-F 0 "#PWR034" H 2500 4660 50  0001 L CNN
+F 0 "#PWR112" H 2500 4660 50  0001 L CNN
 F 1 "3v3" H 2500 4640 50  0000 C CNN
 F 2 "" H 2500 4550 60  0001 C CNN
@@
 $EndComp
 $Comp
-L GND #PWR035
+L GND #PWR110
 U 1 1 585BB030
 P 2400 4650
-F 0 "#PWR035" H 2270 4690 50  0001 L CNN
+F 0 "#PWR110" H 2270 4690 50  0001 L CNN
 F 1 "GND" H 2400 4550 50  0000 C CNN
 F 2 "" H 2400 4650 60  0001 C CNN
@@
 LED1
 $Comp
-L GND #PWR036
+L GND #PWR115
 U 1 1 585146B8
 P 11450 8800
-F 0 "#PWR036" H 11320 8840 50  0001 L CNN
+F 0 "#PWR115" H 11320 8840 50  0001 L CNN
 F 1 "GND" H 11450 8700 50  0000 C CNN
 F 2 "" H 11450 8800 60  0001 C CNN
@@
 LED2
 $Comp
-L GND #PWR037
+L GND #PWR116
 U 1 1 58514E45
 P 11450 9100
-F 0 "#PWR037" H 11320 9140 50  0001 L CNN
+F 0 "#PWR116" H 11320 9140 50  0001 L CNN
 F 1 "GND" H 11450 9000 50  0000 C CNN
 F 2 "" H 11450 9100 60  0001 C CNN
@@
 LED3
 $Comp
-L GND #PWR038
+L GND #PWR117
 U 1 1 58515766
 P 11450 9400
-F 0 "#PWR038" H 11320 9440 50  0001 L CNN
+F 0 "#PWR117" H 11320 9440 50  0001 L CNN
 F 1 "GND" H 11450 9300 50  0000 C CNN
 F 2 "" H 11450 9400 60  0001 C CNN

Commit message: 22 airwires to go
Parts:
- removed C123: 100n, agg:0603, symbol C
- removed D104: USBLC6-2P6, agg:SOT-666, symbol USBLC6-2P6
- removed J101: MICROUSB, agg:MICROUSB_MOLEX_47589-0001, symbol MICROUSB
- removed P102: SWD_TC, agg:TC2030-NL, symbol SWD_TC
- removed R109: 10k, agg:0603, symbol R
Connections:
- net USB_D- is gone; now on net ~CE: IC101.75 (PB14)
- net VUSB is gone; now on net ~PGOOD: IC101.74 (PB13)
- net CS2100_SDA: now also IC101.99 (PC9); no longer IC101.55 (PF15)
- net LED1: now also IC101.135 (PB5); no longer IC101.87 (PG2)
- net LED2: now also IC101.136 (PB6); no longer IC101.88 (PG3)
- net LED3: now also IC101.137 (PB7); no longer IC101.89 (PG4)
- net SD2100_SCL: now also IC101.100 (PA8); no longer IC101.54 (PF14)
- net ~CE: no longer IC101.10 (PF0)
- net ~CHG: now also IC101.73 (PB12); no longer IC101.12 (PF2)
- net ~PGOOD: no longer IC101.11 (PF1)
- net USB_D+: no longer names the net of IC101.76 (PB15)
Other:
- note removed: "USB Connector"
- moved on the sheet: D101, D102, D103, P101, R101, R102, R103

Commit message: cleaned up all the fast lines
Connections:
- net PHY_~RST: now reaches IC101.76 (PB15)
- no-connect marks 50 -> 49

Commit message: add farnell part numbers for passives
Parts:
- C101, C102, C105, C106, C107, C108, C109, C110, C111, C112, C113, C114, C115, C116, C119: Farnell (none) -> 1759037
- C103: Farnell (none) -> 2320818
- C104, C120, C122: Farnell (none) -> 1759407
- C117, C118: Farnell (none) -> 2320817
- C121: Farnell (none) -> 1759102
- D101: Farnell (none) -> 2290329
- D102: Farnell (none) -> 2290330
- D103: Farnell (none) -> 2290328
- R101, R102, R103: Farnell (none) -> 9330380
- R104, R105, R106, R107, R108: Farnell (none) -> 9331255
