File: hardware/linetime_battery.sch (KiCad schematic (older format))
At the start: 0 parts

Commit message: schematic basically done...
Parts:
- added C501, C502, C503: 4µ7, agg:0603, symbol C
- added IC501: BQ24232HA, agg:QFN-16-EP-TI, symbol BQ24232HA
- added J501: BATT, agg:B02B-PASK, symbol CONN_01x02
- added R501: 4k32, agg:0603, symbol R
- added R502: DNS, agg:0603, symbol R
- added R503: 10k, agg:0603, symbol R
- added R504, R505: 100k, agg:0603, symbol R
Connections:
- new net: IC501.1 (TS), R503.2
- new net: IC501.14 (TMR), R502.2
- new net: C503.1, IC501.2 (BAT), IC501.3 (BAT), J501.2, R504.1
- new net DC_IN: C501.1, IC501.13 (IN)
- new net DC_OUT: C502.1, IC501.10 (OUT), IC501.11 (OUT), IC501.6 (EN1)
- new net GND: C501.2, C502.2, C503.2, IC501.5 (EN2), IC501.8 (VSS), IC501.EP (VSS), J501.1, R501.1, R502.1, R503.1, R505.2
- new net I_CHG: IC501.16 (ISET), R501.2
- new net V_BATT/2: R504.2, R505.1
- new net ~CE: IC501.4 (~CE)
- new net ~CHG: IC501.9 (~CHG)
- new net ~PGOOD: IC501.7 (~PGOOD)
- no-connect marks 0 -> 2

Commit message: WIP routing
Parts:
- J501: footprint agg:B02B-PASK -> agg:S02B-PASK-2
Connections:
- net V_BATT/2 renamed V_BATT_MON
Changed lines of the file:
@@
 F 0 "J501" H 6500 3900 50  0000 L CNN
 F 1 "BATT" V 6450 3750 50  0000 C CNN
-F 2 "agg:B02B-PASK" H 6550 3800 50  0001 C CNN
+F 2 "agg:S02B-PASK-2" H 6550 3800 50  0001 C CNN
 F 3 "" H 6550 3800 50  0001 C CNN
 	1    6550 3800
@@
 Connection ~ 5700 3700
 $Comp
-L GND #PWR0106
+L GND #PWR502
 U 1 1 584C0C58
 P 4450 3350
-F 0 "#PWR0106" H 4320 3390 50  0001 L CNN
+F 0 "#PWR502" H 4320 3390 50  0001 L CNN
 F 1 "GND" H 4450 3250 50  0000 C CNN
 F 2 "" H 4450 3350 60  0001 C CNN
@@
 Connection ~ 4450 3300
 $Comp
-L GND #PWR0107
+L GND #PWR506
 U 1 1 584C0C96
 P 6150 3900
-F 0 "#PWR0107" H 6020 3940 50  0001 L CNN
+F 0 "#PWR506" H 6020 3940 50  0001 L CNN
 F 1 "GND" H 6150 3800 50  0000 C CNN
 F 2 "" H 6150 3900 60  0001 C CNN
@@
 Connection ~ 6150 3700
 $Comp
-L GND #PWR0108
+L GND #PWR507
 U 1 1 584C0CEB
 P 6400 3850
-F 0 "#PWR0108" H 6270 3890 50  0001 L CNN
+F 0 "#PWR507" H 6270 3890 50  0001 L CNN
 F 1 "GND" H 6400 3750 50  0000 C CNN
 F 2 "" H 6400 3850 60  0001 C CNN
@@
 $EndComp
 $Comp
-L GND #PWR0109
+L GND #PWR501
 U 1 1 584C13B1
 P 4300 4150
-F 0 "#PWR0109" H 4170 4190 50  0001 L CNN
+F 0 "#PWR501" H 4170 4190 50  0001 L CNN
 F 1 "GND" H 4300 4050 50  0000 C CNN
 F 2 "" H 4300 4150 60  0001 C CNN
@@
 Connection ~ 6050 3100
 $Comp
-L GND #PWR0110
+L GND #PWR505
 U 1 1 584C18CE
 P 6050 3300
-F 0 "#PWR0110" H 5920 3340 50  0001 L CNN
+F 0 "#PWR505" H 5920 3340 50  0001 L CNN
 F 1 "GND" H 6050 3200 50  0000 C CNN
 F 2 "" H 6050 3300 60  0001 C CNN
@@
 NoConn ~ 4650 3600
 $Comp
-L GND #PWR0111
+L GND #PWR503
 U 1 1 584C310A
 P 5750 3500
-F 0 "#PWR0111" H 5620 3540 50  0001 L CNN
+F 0 "#PWR503" H 5620 3540 50  0001 L CNN
 F 1 "GND" H 5750 3400 50  0000 C CNN
 F 2 "" H 5750 3500 60  0001 C CNN
@@
 Connection ~ 6350 3700
 Text HLabel 6950 3750 2    40   Output ~ 0
-V_BATT/2
+V_BATT_MON
 $Comp
 L R R504
@@
 $EndComp
 $Comp
-L GND #PWR0112
+L GND #PWR508
 U 1 1 584C4401
 P 6850 3950
-F 0 "#PWR0112" H 6720 3990 50  0001 L CNN
+F 0 "#PWR508" H 6720 3990 50  0001 L CNN
 F 1 "GND" H 6850 3850 50  0000 C CNN
 F 2 "" H 6850 3950 60  0001 C CNN
@@
 $EndComp
 $Comp
-L GND #PWR0113
+L GND #PWR504
 U 1 1 584C4C07
 P 5850 3900
-F 0 "#PWR0113" H 5720 3940 50  0001 L CNN
+F 0 "#PWR504" H 5720 3940 50  0001 L CNN
 F 1 "GND" H 5850 3800 50  0000 C CNN
 F 2 "" H 5850 3900 60  0001 C CNN

Commit message: add farnell part numbers for passives
Parts:
- C501, C502, C503: Farnell (none) -> 2320818
- R501: Farnell (none) -> 2074263
- R503: Farnell (none) -> 9330399
- R504, R505: value 100k -> 110k; Farnell (none) -> 9330461
Changed lines of the file:
@@
 F 2 "agg:0603" H 6150 3750 50  0001 C CNN
 F 3 "" H 6150 3750 50  0001 C CNN
+F 4 "2320818" H 6150 3750 60  0001 C CNN "Farnell"
 	1    6150 3750
 	0    1    1    0
@@
 Connection ~ 5700 3700
 $Comp
-L GND #PWR502
+L GND #PWR0101
 U 1 1 584C0C58
 P 4450 3350
-F 0 "#PWR502" H 4320 3390 50  0001 L CNN
+F 0 "#PWR0101" H 4320 3390 50  0001 L CNN
 F 1 "GND" H 4450 3250 50  0000 C CNN
 F 2 "" H 4450 3350 60  0001 C CNN
@@
 Connection ~ 4450 3300
 $Comp
-L GND #PWR506
+L GND #PWR0102
 U 1 1 584C0C96
 P 6150 3900
-F 0 "#PWR506" H 6020 3940 50  0001 L CNN
+F 0 "#PWR0102" H 6020 3940 50  0001 L CNN
 F 1 "GND" H 6150 3800 50  0000 C CNN
 F 2 "" H 6150 3900 60  0001 C CNN
@@
 Connection ~ 6150 3700
 $Comp
-L GND #PWR507
+L GND #PWR0103
 U 1 1 584C0CEB
 P 6400 3850
-F 0 "#PWR507" H 6270 3890 50  0001 L CNN
+F 0 "#PWR0103" H 6270 3890 50  0001 L CNN
 F 1 "GND" H 6400 3750 50  0000 C CNN
 F 2 "" H 6400 3850 60  0001 C CNN
@@
 F 2 "agg:0603" H 4400 3700 50  0001 C CNN
 F 3 "" H 4400 3700 50  0001 C CNN
+F 4 "2074263" H 4400 3700 60  0001 C CNN "Farnell"
 	1    4400 3700
 	1    0    0    -1
 $EndComp
 $Comp
-L GND #PWR501
+L GND #PWR0104
 U 1 1 584C13B1
 P 4300 4150
-F 0 "#PWR501" H 4170 4190 50  0001 L CNN
+F 0 "#PWR0104" H 4170 4190 50  0001 L CNN
 F 1 "GND" H 4300 4050 50  0000 C CNN
 F 2 "" H 4300 4150 60  0001 C CNN
@@
 F 2 "agg:0603" H 6050 3150 50  0001 C CNN
 F 3 "" H 6050 3150 50  0001 C CNN
+F 4 "2320818" H 6050 3150 60  0001 C CNN "Farnell"
 	1    6050 3150
 	0    1    1    0
@@
 Connection ~ 6050 3100
 $Comp
-L GND #PWR505
+L GND #PWR0105
 U 1 1 584C18CE
 P 6050 3300
-F 0 "#PWR505" H 5920 3340 50  0001 L CNN
+F 0 "#PWR0105" H 5920 3340 50  0001 L CNN
 F 1 "GND" H 6050 3200 50  0000 C CNN
 F 2 "" H 6050 3300 60  0001 C CNN
@@
 NoConn ~ 4650 3600
 $Comp
-L GND #PWR503
+L GND #PWR0106
 U 1 1 584C310A
 P 5750 3500
-F 0 "#PWR503" H 5620 3540 50  0001 L CNN
+F 0 "#PWR0106" H 5620 3540 50  0001 L CNN
 F 1 "GND" H 5750 3400 50  0000 C CNN
 F 2 "" H 5750 3500 60  0001 C CNN
@@
 P 6850 3600
 F 0 "R504" H 6900 3650 50  0000 C CNN
-F 1 "100k" H 6900 3550 50  0000 C CNN
+F 1 "110k" H 6900 3550 50  0000 C CNN
 F 2 "agg:0603" H 6850 3600 50  0001 C CNN
 F 3 "" H 6850 3600 50  0001 C CNN
+F 4 "9330461" H 6850 3600 60  0001 C CNN "Farnell"
 	1    6850 3600
 	0    1    1    0
@@
 P 6850 3800
 F 0 "R505" H 6900 3850 50  0000 C CNN
-F 1 "100k" H 6900 3750 50  0000 C CNN
+F 1 "110k" H 6900 3750 50  0000 C CNN
 F 2 "agg:0603" H 6850 3800 50  0001 C CNN
 F 3 "" H 6850 3800 50  0001 C CNN
+F 4 "9330461" H 6850 3800 60  0001 C CNN "Farnell"
 	1    6850 3800
 	0    1    1    0
 $EndComp
 $Comp
-L GND #PWR508
+L GND #PWR0107
 U 1 1 584C4401
 P 6850 3950
-F 0 "#PWR508" H 6720 3990 50  0001 L CNN
+F 0 "#PWR0107" H 6720 3990 50  0001 L CNN
 F 1 "GND" H 6850 3850 50  0000 C CNN
 F 2 "" H 6850 3950 60  0001 C CNN
@@
 F 2 "agg:0603" H 5800 3900 50  0001 C CNN
 F 3 "" H 5800 3900 50  0001 C CNN
+F 4 "9330399" H 5800 3900 60  0001 C CNN "Farnell"
 	1    5800 3900
 	-1   0    0    1
 $EndComp
 $Comp
-L GND #PWR504
+L GND #PWR0108
 U 1 1 584C4C07
 P 5850 3900
-F 0 "#PWR504" H 5720 3940 50  0001 L CNN
+F 0 "#PWR0108" H 5720 3940 50  0001 L CNN
 F 1 "GND" H 5850 3800 50  0000 C CNN
 F 2 "" H 5850 3900 60  0001 C CNN
@@
 F 2 "agg:0603" H 4450 3150 50  0001 C CNN
 F 3 "" H 4450 3150 50  0001 C CNN
+F 4 "2320818" H 4450 3150 60  0001 C CNN "Farnell"
 	1    4450 3150
 	0    1    1    0
