File: hardware/linetime_ethernet.sch (KiCad schematic (older format))
At the start: 79 parts

Commit message: schematic basically done...
Parts:
- removed C? (x4): 10n 200V, agg:0805, symbol C
- removed C? (x9): 1n 2kV, agg:0805, symbol C
- removed C? (x2): 100n, agg:0603, symbol C
- removed C? (x2): 47µ, symbol C
- removed C? (x3): 1µ, symbol C
- removed C?: 12µ, symbol C
- removed C?: 470p, agg:0603, symbol C
- removed C?: 1000µ, symbol CP
- removed C?: 15n, agg:0603, symbol C
- removed C?: 3n3, agg:0603, symbol C
- removed D? (x2): LED, symbol LED
- removed D?: 1N4148, agg:SOD-323, symbol D
- removed D?: DFLT30A-7, symbol D
- removed D?: PDS1040, symbol SCHOTTKY
- removed IC?: Si3402-B, agg:QFN-20-EP-SI3402-B, symbol Si3402-B
- removed IC?: TLV431, agg:SOT-23, symbol TLV431
- removed IC?: VO618A, agg:VO618A-SMD-4-7, symbol VO618A
- removed J?: 8P8C, symbol CONN_01x08
- removed L? (x4): FB, symbol L
- removed L?: 1µ, symbol L
- removed R? (x3): 75, agg:0603, symbol R
- removed R?: 24.3k, agg:0603, symbol R
- removed R?: 47k, symbol R
- removed R?: 10, agg:0603, symbol R
- removed R? (x2): 0, symbol R
- removed R?: 4k99, symbol R
- removed R?: 2k05, symbol R
- removed R?: 36k5, symbol R
- removed R?: 12k1, symbol R
- removed T?: FA2672, agg:FA267x, symbol FA267x
- added IC401: RJHSE-5381, agg:RJHSE-538X, symbol RJHSE-538x
- L401: renamed from L?; footprint (none) -> agg:0603; Farnell (none) -> 1669708
- Y401: renamed from Y?; footprint (none) -> agg:XTAL-50x32; Farnell (none) -> 2101328
- gave numbers to parts that had none: 25
Connections:
- net CT1: now also R402.1
- net CT2: now also R403.1
- net GND: now also IC401.S (SHIELD)
- net at T401.1 (TD+): now also IC401.6 (RX-)
- net at T401.3 (TD-): now also IC401.3 (RX+)
- net at T401.6 (RD+): now also IC401.2 (TX-)
- net at T401.8 (RD-): now also IC401.1 (TX+)
- net LINK_LED: now reaches IC402.23 (LED0)
- net LINK_LED: now also IC401.9 (LED1_C)
- net at R401.1: now also IC401.10 (LED1_A)
- net TXDO0 renamed TXD0
- no-connect marks 3 -> 8
Other:
- note added: "Bob Smith terminations"
- note removed: "ADD SHIELD CONNECTION"
- note removed: "Isolated PoE 5V SMPS"
- note removed: "Modified Bob Smith terminations"
- note removed: "To-Do:\n* Check SMPS output capacitors are correct\n* Read through SMPS app note carefully\n* Use ethernet jack with LEDs"
- note removed: "USE CONNECTOR WITH LEDS"
- moved on the sheet: C401, C402, C403, C404, C405, C406, C407, C408, C409, C410, C411, C412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

Commit message: 22 airwires to go
Parts:
- C401: footprint agg:0805 -> agg:1206; Farnell (none) -> 1855909
Changed lines of the file:
@@
 EESchema Schematic File Version 2
-LIBS:agg-kicad
 LIBS:linetime-cache
 EELAYER 25 0
@@
 $EndComp
 $Comp
-L 3v3 #PWR405
+L 3v3 #PWR088
 U 1 1 584B9E07
 P 4750 2500
-F 0 "#PWR405" H 4750 2610 50  0001 L CNN
+F 0 "#PWR088" H 4750 2610 50  0001 L CNN
 F 1 "3v3" H 4750 2590 50  0000 C CNN
 F 2 "" H 4750 2500 60  0001 C CNN
@@
 $EndComp
 $Comp
-L 3v3 #PWR417
+L 3v3 #PWR089
 U 1 1 584B9E72
 P 8250 3600
-F 0 "#PWR417" H 8250 3710 50  0001 L CNN
+F 0 "#PWR089" H 8250 3710 50  0001 L CNN
 F 1 "3v3" H 8250 3690 50  0000 C CNN
 F 2 "" H 8250 3600 60  0001 C CNN
@@
 $EndComp
 $Comp
-L GND #PWR419
+L GND #PWR090
 U 1 1 584BA2FE
 P 8500 4550
-F 0 "#PWR419" H 8370 4590 50  0001 L CNN
+F 0 "#PWR090" H 8370 4590 50  0001 L CNN
 F 1 "GND" H 8500 4450 50  0000 C CNN
 F 2 "" H 8500 4550 60  0001 C CNN
@@
 $EndComp
 $Comp
-L 3v3 #PWR418
+L 3v3 #PWR091
 U 1 1 584BA361
 P 8500 4100
-F 0 "#PWR418" H 8500 4210 50  0001 L CNN
+F 0 "#PWR091" H 8500 4210 50  0001 L CNN
 F 1 "3v3" H 8500 4190 50  0000 C CNN
 F 2 "" H 8500 4100 60  0001 C CNN
@@
 $EndComp
 $Comp
-L GND #PWR412
+L GND #PWR092
 U 1 1 584BAE67
 P 5500 4200
-F 0 "#PWR412" H 5370 4240 50  0001 L CNN
+F 0 "#PWR092" H 5370 4240 50  0001 L CNN
 F 1 "GND" H 5500 4100 50  0000 C CNN
 F 2 "" H 5500 4200 60  0001 C CNN
@@
 $EndComp
 $Comp
-L GND #PWR415
+L GND #PWR093
 U 1 1 584BB204
 P 6100 3500
-F 0 "#PWR415" H 5970 3540 50  0001 L CNN
+F 0 "#PWR093" H 5970 3540 50  0001 L CNN
 F 1 "GND" H 6100 3400 50  0000 C CNN
 F 2 "" H 6100 3500 60  0001 C CNN
@@
 $EndComp
 $Comp
-L GND #PWR404
+L GND #PWR094
 U 1 1 584BC166
 P 4500 2900
-F 0 "#PWR404" H 4370 2940 50  0001 L CNN
+F 0 "#PWR094" H 4370 2940 50  0001 L CNN
 F 1 "GND" H 4500 2800 50  0000 C CNN
 F 2 "" H 4500 2900 60  0001 C CNN
@@
 $EndComp
 $Comp
-L GND #PWR414
+L GND #PWR095
 U 1 1 584BC26D
 P 5900 3350
-F 0 "#PWR414" H 5770 3390 50  0001 L CNN
+F 0 "#PWR095" H 5770 3390 50  0001 L CNN
 F 1 "GND" H 5900 3250 50  0000 C CNN
 F 2 "" H 5900 3350 60  0001 C CNN
@@
 $EndComp
 $Comp
-L GND #PWR413
+L GND #PWR096
 U 1 1 584BC2B7
 P 5650 3350
-F 0 "#PWR413" H 5520 3390 50  0001 L CNN
+F 0 "#PWR096" H 5520 3390 50  0001 L CNN
 F 1 "GND" H 5650 3250 50  0000 C CNN
 F 2 "" H 5650 3350 60  0001 C CNN
@@
 $EndComp
 $Comp
-L GND #PWR406
+L GND #PWR097
 U 1 1 584BC475
 P 4750 2900
-F 0 "#PWR406" H 4620 2940 50  0001 L CNN
+F 0 "#PWR097" H 4620 2940 50  0001 L CNN
 F 1 "GND" H 4750 2800 50  0000 C CNN
 F 2 "" H 4750 2900 60  0001 C CNN
@@
 $EndComp
 $Comp
-L PWR #FLG401
+L PWR #FLG098
 U 1 1 584BC5A0
 P 4500 2650
-F 0 "#FLG401" H 4500 2810 50  0001 C CNN
+F 0 "#FLG098" H 4500 2810 50  0001 C CNN
 F 1 "PWR" H 4500 2740 50  0000 C CNN
 F 2 "" H 4500 2650 50  0001 C CNN
@@
 $EndComp
 $Comp
-L GND #PWR410
+L GND #PWR099
 U 1 1 584BCAA1
 P 5100 3150
-F 0 "#PWR410" H 4970 3190 50  0001 L CNN
+F 0 "#PWR099" H 4970 3190 50  0001 L CNN
 F 1 "GND" H 5100 3050 50  0000 C CNN
 F 2 "" H 5100 3150 60  0001 C CNN
@@
 $EndComp
 $Comp
-L GND #PWR411
+L GND #PWR0100
 U 1 1 584BCAA8
 P 5350 3150
-F 0 "#PWR411" H 5220 3190 50  0001 L CNN
+F 0 "#PWR0100" H 5220 3190 50  0001 L CNN
 F 1 "GND" H 5350 3050 50  0000 C CNN
 F 2 "" H 5350 3150 60  0001 C CNN
@@
 $EndComp
 $Comp
-L 3v3 #PWR409
+L 3v3 #PWR0101
 U 1 1 584BCC0A
 P 5050 2900
-F 0 "#PWR409" H 5050 3010 50  0001 L CNN
+F 0 "#PWR0101" H 5050 3010 50  0001 L CNN
 F 1 "3v3" H 5050 2990 50  0000 C CNN
 F 2 "" H 5050 2900 60  0001 C CNN
@@
 $EndComp
 $Comp
-L GND #PWR407
+L GND #PWR0102
 U 1 1 584BDBA9
 P 4750 3600
-F 0 "#PWR407" H 4620 3640 50  0001 L CNN
+F 0 "#PWR0102" H 4620 3640 50  0001 L CNN
 F 1 "GND" H 4750 3500 50  0000 C CNN
 F 2 "" H 4750 3600 60  0001 C CNN
@@
 $EndComp
 $Comp
-L GND #PWR408
+L GND #PWR0103
 U 1 1 584BDCAE
 P 4750 4000
-F 0 "#PWR408" H 4620 4040 50  0001 L CNN
+F 0 "#PWR0103" H 4620 4040 50  0001 L CNN
 F 1 "GND" H 4750 3900 50  0000 C CNN
 F 2 "" H 4750 4000 60  0001 C CNN
@@
 CT2
 $Comp
-L GND #PWR416
+L GND #PWR0104
 U 1 1 584C02A5
 P 7600 4050
-F 0 "#PWR416" H 7470 4090 50  0001 L CNN
+F 0 "#PWR0104" H 7470 4090 50  0001 L CNN
 F 1 "GND" H 7600 3950 50  0000 C CNN
 F 2 "" H 7600 4050 60  0001 C CNN
@@
 $EndComp
 $Comp
-L 3v3 #PWR401
+L 3v3 #PWR0105
 U 1 1 584C07D6
 P 1550 3450
-F 0 "#PWR401" H 1550 3560 50  0001 L CNN
+F 0 "#PWR0105" H 1550 3560 50  0001 L CNN
 F 1 "3v3" H 1550 3540 50  0000 C CNN
 F 2 "" H 1550 3450 60  0001 C CNN
@@
 F 0 "C401" H 2950 5170 50  0000 C CNN
 F 1 "1n 2kV" H 2950 5030 50  0000 C CNN
-F 2 "agg:0805" H 2900 5100 50  0001 C CNN
+F 2 "agg:1206" H 2900 5100 50  0001 C CNN
 F 3 "" H 2900 5100 50  0001 C CNN
+F 4 "1855909" H 2900 5100 60  0001 C CNN "Farnell"
 	1    2900 5100
 	-1   0    0    1
 $EndComp
 $Comp
-L GND #PWR403
+L GND #PWR0106
 U 1 1 584C57B0
 P 2750 5150
-F 0 "#PWR403" H 2620 5190 50  0001 L CNN
+F 0 "#PWR0106" H 2620 5190 50  0001 L CNN
 F 1 "GND" H 2750 5050 50  0000 C CNN
 F 2 "" H 2750 5150 60  0001 C CNN
@@
 $EndComp
 $Comp
-L GND #PWR402
+L GND #PWR0107
 U 1 1 584B6EFC
 P 2050 4050
-F 0 "#PWR402" H 1920 4090 50  0001 L CNN
+F 0 "#PWR0107" H 1920 4090 50  0001 L CNN
 F 1 "GND" H 2050 3950 50  0000 C CNN
 F 2 "" H 2050 4050 60  0001 C CNN

Commit message: cleaned up all the fast lines
Parts:
- removed C412: 10µ, agg:0603, symbol C
- removed D401: 1N4148, agg:SOD-323, symbol D
- added R411, R412, R413: 33, agg:0603, symbol R
Connections:
- net 3v3: no longer R410.1
- net GND: now also R410.2
- net TXD0: now also R413.2; no longer IC402.20 (TXD0)
- net TXD1: now also R412.2; no longer IC402.21 (TXD1)
- net TXEN: now also R411.2; no longer IC402.19 (TXEN)
- net PHY_~RST: now reaches IC402.24 (~RST)
- net PHY_~RST: now also R410.1; no longer R410.2
- new net: IC402.19 (TXEN), R411.1
- new net: IC402.20 (TXD0), R413.1
- new net: IC402.21 (TXD1), R412.1
Other:
- note added: "Series resistors placed\nnear that signal's transmitter:\nRX*, CRS_DV, REF_CLK near PHY,\nTX* near MAC"
- moved on the sheet: R410
Changed lines of the file:
@@
 EESchema Schematic File Version 2
+LIBS:agg-kicad
 LIBS:linetime-cache
 EELAYER 25 0
@@
 $EndComp
 $Comp
-L 3v3 #PWR088
+L 3v3 #PWR405
 U 1 1 584B9E07
 P 4750 2500
-F 0 "#PWR088" H 4750 2610 50  0001 L CNN
+F 0 "#PWR405" H 4750 2610 50  0001 L CNN
 F 1 "3v3" H 4750 2590 50  0000 C CNN
 F 2 "" H 4750 2500 60  0001 C CNN
@@
 $EndComp
 $Comp
-L 3v3 #PWR089
+L 3v3 #PWR418
 U 1 1 584B9E72
 P 8250 3600
-F 0 "#PWR089" H 8250 3710 50  0001 L CNN
+F 0 "#PWR418" H 8250 3710 50  0001 L CNN
 F 1 "3v3" H 8250 3690 50  0000 C CNN
 F 2 "" H 8250 3600 60  0001 C CNN
@@
 $EndComp
 $Comp
-L D D401
-U 1 1 584B9F3E
-P 8400 4200
-F 0 "D401" H 8450 4270 50  0000 C CNN
-F 1 "1N4148" H 8450 4130 50  0000 C CNN
-F 2 "agg:SOD-323" H 8400 4200 50  0001 C CNN
-F 3 "" H 8400 4200 50  0001 C CNN
-F 4 "1466524" H 8400 4200 60  0001 C CNN "Farnell"
-	1    8400 4200
-	0    1    1    0
-$EndComp
-$Comp
 L R R410
 U 1 1 584B9FA9
-P 8600 4200
-F 0 "R410" H 8650 4250 50  0000 C CNN
-F 1 "10k" H 8650 4150 50  0000 C CNN
-F 2 "agg:0603" H 8600 4200 50  0001 C CNN
-F 3 "" H 8600 4200 50  0001 C CNN
-	1    8600 4200
+P 7500 4450
+F 0 "R410" H 7550 4500 50  0000 C CNN
+F 1 "10k" H 7550 4400 50  0000 C CNN
+F 2 "agg:0603" H 7500 4450 50  0001 C CNN
+F 3 "" H 7500 4450 50  0001 C CNN
+	1    7500 4450
 	0    1    1    0
 $EndComp
 $Comp
-L C C412
-U 1 1 584BA030
-P 8500 4400
-F 0 "C412" H 8550 4470 50  0000 C CNN
-F 1 "10µ" H 8550 4330 50  0000 C CNN
-F 2 "agg:0603" H 8500 4400 50  0001 C CNN
-F 3 "" H 8500 4400 50  0001 C CNN
-	1    8500 4400
-	0    1    1    0
-$EndComp
-$Comp
-L GND #PWR090
+L GND #PWR416
 U 1 1 584BA2FE
-P 8500 4550
-F 0 "#PWR090" H 8370 4590 50  0001 L CNN
-F 1 "GND" H 8500 4450 50  0000 C CNN
-F 2 "" H 8500 4550 60  0001 C CNN
-F 3 "" H 8500 4550 60  0001 C CNN
-	1    8500 4550
-	1    0    0    -1
-$EndComp
-$Comp
-L 3v3 #PWR091
-U 1 1 584BA361
-P 8500 4100
-F 0 "#PWR091" H 8500 4210 50  0001 L CNN
-F 1 "3v3" H 8500 4190 50  0000 C CNN
-F 2 "" H 8500 4100 60  0001 C CNN
-F 3 "" H 8500 4100 60  0001 C CNN
-	1    8500 4100
+P 7500 4600
+F 0 "#PWR416" H 7370 4640 50  0001 L CNN
+F 1 "GND" H 7500 4500 50  0000 C CNN
+F 2 "" H 7500 4600 60  0001 C CNN
+F 3 "" H 7500 4600 60  0001 C CNN
+	1    7500 4600
 	1    0    0    -1
 $EndComp
@@
 $EndComp
 $Comp
-L GND #PWR092
+L GND #PWR412
 U 1 1 584BAE67
 P 5500 4200
-F 0 "#PWR092" H 5370 4240 50  0001 L CNN
+F 0 "#PWR412" H 5370 4240 50  0001 L CNN
 F 1 "GND" H 5500 4100 50  0000 C CNN
 F 2 "" H 5500 4200 60  0001 C CNN
@@
 $EndComp
 $Comp
-L GND #PWR093
+L GND #PWR415
 U 1 1 584BB204
 P 6100 3500
-F 0 "#PWR093" H 5970 3540 50  0001 L CNN
+F 0 "#PWR415" H 5970 3540 50  0001 L CNN
 F 1 "GND" H 6100 3400 50  0000 C CNN
 F 2 "" H 6100 3500 60  0001 C CNN
@@
 $EndComp
 $Comp
-L GND #PWR094
+L GND #PWR404
 U 1 1 584BC166
 P 4500 2900
-F 0 "#PWR094" H 4370 2940 50  0001 L CNN
+F 0 "#PWR404" H 4370 2940 50  0001 L CNN
 F 1 "GND" H 4500 2800 50  0000 C CNN
 F 2 "" H 4500 2900 60  0001 C CNN
@@
 $EndComp
 $Comp
-L GND #PWR095
+L GND #PWR414
 U 1 1 584BC26D
 P 5900 3350
-F 0 "#PWR095" H 5770 3390 50  0001 L CNN
+F 0 "#PWR414" H 5770 3390 50  0001 L CNN
 F 1 "GND" H 5900 3250 50  0000 C CNN
 F 2 "" H 5900 3350 60  0001 C CNN
@@
 $EndComp
 $Comp
-L GND #PWR096
+L GND #PWR413
 U 1 1 584BC2B7
 P 5650 3350
-F 0 "#PWR096" H 5520 3390 50  0001 L CNN
+F 0 "#PWR413" H 5520 3390 50  0001 L CNN
 F 1 "GND" H 5650 3250 50  0000 C CNN
 F 2 "" H 5650 3350 60  0001 C CNN
@@
 $EndComp
 $Comp
-L GND #PWR097
+L GND #PWR406
 U 1 1 584BC475
 P 4750 2900
-F 0 "#PWR097" H 4620 2940 50  0001 L CNN
+F 0 "#PWR406" H 4620 2940 50  0001 L CNN
 F 1 "GND" H 4750 2800 50  0000 C CNN
 F 2 "" H 4750 2900 60  0001 C CNN
@@
 $EndComp
 $Comp
-L PWR #FLG098
+L PWR #FLG401
 U 1 1 584BC5A0
 P 4500 2650
-F 0 "#FLG098" H 4500 2810 50  0001 C CNN
+F 0 "#FLG401" H 4500 2810 50  0001 C CNN
 F 1 "PWR" H 4500 2740 50  0000 C CNN
 F 2 "" H 4500 2650 50  0001 C CNN
@@
 $EndComp
 $Comp
-L GND #PWR099
+L GND #PWR410
 U 1 1 584BCAA1
 P 5100 3150
-F 0 "#PWR099" H 4970 3190 50  0001 L CNN
+F 0 "#PWR410" H 4970 3190 50  0001 L CNN
 F 1 "GND" H 5100 3050 50  0000 C CNN
 F 2 "" H 5100 3150 60  0001 C CNN
@@
 $EndComp
 $Comp
-L GND #PWR0100
+L GND #PWR411
 U 1 1 584BCAA8
 P 5350 3150
-F 0 "#PWR0100" H 5220 3190 50  0001 L CNN
+F 0 "#PWR411" H 5220 3190 50  0001 L CNN
 F 1 "GND" H 5350 3050 50  0000 C CNN
 F 2 "" H 5350 3150 60  0001 C CNN
@@
 $EndComp
 $Comp
-L 3v3 #PWR0101
+L 3v3 #PWR409
 U 1 1 584BCC0A
 P 5050 2900
-F 0 "#PWR0101" H 5050 3010 50  0001 L CNN
+F 0 "#PWR409" H 5050 3010 50  0001 L CNN
 F 1 "3v3" H 5050 2990 50  0000 C CNN
 F 2 "" H 5050 2900 60  0001 C CNN
@@
 $EndComp
 $Comp
-L GND #PWR0102
+L GND #PWR407
 U 1 1 584BDBA9
 P 4750 3600
-F 0 "#PWR0102" H 4620 3640 50  0001 L CNN
+F 0 "#PWR407" H 4620 3640 50  0001 L CNN
 F 1 "GND" H 4750 3500 50  0000 C CNN
 F 2 "" H 4750 3600 60  0001 C CNN
@@
 $EndComp
 $Comp
-L GND #PWR0103
+L GND #PWR408
 U 1 1 584BDCAE
 P 4750 4000
-F 0 "#PWR0103" H 4620 4040 50  0001 L CNN
+F 0 "#PWR408" H 4620 4040 50  0001 L CNN
 F 1 "GND" H 4750 3900 50  0000 C CNN
 F 2 "" H 4750 4000 60  0001 C CNN
@@
 CT2
 $Comp
-L GND #PWR0104
+L GND #PWR417
 U 1 1 584C02A5
 P 7600 4050
-F 0 "#PWR0104" H 7470 4090 50  0001 L CNN
+F 0 "#PWR417" H 7470 4090 50  0001 L CNN
 F 1 "GND" H 7600 3950 50  0000 C CNN
 F 2 "" H 7600 4050 60  0001 C CNN
@@
 $EndComp
 $Comp
-L 3v3 #PWR0105
+L 3v3 #PWR401
 U 1 1 584C07D6
 P 1550 3450
-F 0 "#PWR0105" H 1550 3560 50  0001 L CNN
+F 0 "#PWR401" H 1550 3560 50  0001 L CNN
 F 1 "3v3" H 1550 3540 50  0000 C CNN
 F 2 "" H 1550 3450 60  0001 C CNN
@@
 $EndComp
 $Comp
-L GND #PWR0106
+L GND #PWR403
 U 1 1 584C57B0
 P 2750 5150
-F 0 "#PWR0106" H 2620 5190 50  0001 L CNN
+F 0 "#PWR403" H 2620 5190 50  0001 L CNN
 F 1 "GND" H 2750 5050 50  0000 C CNN
 F 2 "" H 2750 5150 60  0001 C CNN
@@
 	7700 3150 7800 3150
 Wire Wire Line
-	7350 3350 7800 3350
-Wire Wire Line
-	7350 3450 7800 3450
-Wire Wire Line
-	7350 3550 7800 3550
-Wire Wire Line
 	7350 3750 7800 3750
 Wire Wire Line
@@
 	8250 3650 8250 3600
 Wire Wire Line
-	7350 4350 8600 4350
-Wire Wire Line
-	8600 4350 8600 4300
-Wire Wire Line
-	8500 4400 8500 4350
-Connection ~ 8500 4350
-Wire Wire Line
-	8400 4350 8400 4300
-Connection ~ 8400 4350
-Wire Wire Line
-	8500 4550 8500 4500
-Wire Wire Line
-	8500 4100 8500 4150
-Wire Wire Line
-	8400 4150 8600 4150
-Wire Wire Line
-	8400 4150 8400 4200
-Wire Wire Line
-	8600 4150 8600 4200
-Connection ~ 8500 4150
+	7500 4600 7500 4550
 Wire Wire Line
 	7350 4250 7500 4250
@@
 $EndComp
 $Comp
-L GND #PWR0107
+L GND #PWR402
 U 1 1 584B6EFC
 P 2050 4050
-F 0 "#PWR0107" H 1920 4090 50  0001 L CNN
+F 0 "#PWR402" H 1920 4090 50  0001 L CNN
 F 1 "GND" H 2050 3950 50  0000 C CNN
 F 2 "" H 2050 4050 60  0001 C CNN
@@
 NoConn ~ 2300 3700
 NoConn ~ 2300 3800
+$Comp
+L R R411
+U 1 1 585723B1
+P 7450 3350
+F 0 "R411" H 7500 3400 50  0000 C CNN
+F 1 "33" H 7500 3300 50  0000 C CNN
+F 2 "agg:0603" H 7450 3350 50  0001 C CNN
+F 3 "" H 7450 3350 50  0001 C CNN
+	1    7450 3350
+	1    0    0    -1
+$EndComp
+$Comp
+L R R413
+U 1 1 58572479
+P 7600 3450
+F 0 "R413" H 7650 3500 50  0000 C CNN
+F 1 "33" H 7650 3400 50  0000 C CNN
+F 2 "agg:0603" H 7600 3450 50  0001 C CNN
+F 3 "" H 7600 3450 50  0001 C CNN
+	1    7600 3450
+	1    0    0    -1
+$EndComp
+$Comp
+L R R412
+U 1 1 585724EB
+P 7450 3550
+F 0 "R412" H 7500 3600 50  0000 C CNN
+F 1 "33" H 7500 3500 50  0000 C CNN
+F 2 "agg:0603" H 7450 3550 50  0001 C CNN
+F 3 "" H 7450 3550 50  0001 C CNN
+	1    7450 3550
+	1    0    0    -1
+$EndComp
+Wire Wire Line
+	7350 3550 7450 3550
+Wire Wire Line
+	7350 3450 7600 3450
+Wire Wire Line
+	7350 3350 7450 3350
+Wire Wire Line
+	7550 3350 7800 3350
+Wire Wire Line
+	7700 3450 7800 3450
+Wire Wire Line
+	7550 3550 7800 3550
+Text Notes 8200 3150 0    40   ~ 0
+Series resistors placed\nnear that signal's transmitter:\nRX*, CRS_DV, REF_CLK near PHY,\nTX* near MAC
+Wire Wire Line
+	7350 4350 7800 4350
+Wire Wire Line
+	7500 4350 7500 4450
+Connection ~ 7500 4350
+Text HLabel 7800 4350 2    40   Input ~ 0
+PHY_~RST
 $EndSCHEMATC
