File: hardware/linetime_ethernet.sch (KiCad schematic (older format))
At the start: 29 parts, among them IC401 RJHSE-5381, IC402 KSZ8081RNx, T401 749013011A, Y401 XTAL

Commit message: add farnell part numbers for passives
Parts:
- C402, C406: Farnell (none) -> 2494232
- C403, C404, C405, C407, C411: Farnell (none) -> 1759037
- C408: Farnell (none) -> 2320817
- C409, C410: Farnell (none) -> 2627466
- R401, R409: Farnell (none) -> 9330380
- R404, R405, R407, R408, R411, R412, R413: Farnell (none) -> 9331050
- R406: Farnell (none) -> 1170871
- R410: Farnell (none) -> 9330399
Changed lines of the file:
@@
 F 2 "agg:0603" H 7450 2850 50  0001 C CNN
 F 3 "" H 7450 2850 50  0001 C CNN
+F 4 "9331050" H 7450 2850 60  0001 C CNN "Farnell"
 	1    7450 2850
 	1    0    0    -1
@@
 F 2 "agg:0603" H 7600 2950 50  0001 C CNN
 F 3 "" H 7600 2950 50  0001 C CNN
+F 4 "9331050" H 7600 2950 60  0001 C CNN "Farnell"
 	1    7600 2950
 	1    0    0    -1
@@
 F 2 "agg:0603" H 7450 3050 50  0001 C CNN
 F 3 "" H 7450 3050 50  0001 C CNN
+F 4 "9331050" H 7450 3050 60  0001 C CNN "Farnell"
 	1    7450 3050
 	1    0    0    -1
@@
 F 2 "agg:0603" H 7600 3150 50  0001 C CNN
 F 3 "" H 7600 3150 50  0001 C CNN
+F 4 "9331050" H 7600 3150 60  0001 C CNN "Farnell"
 	1    7600 3150
 	1    0    0    -1
@@
 F 2 "agg:0603" H 7450 4050 50  0001 C CNN
 F 3 "" H 7450 4050 50  0001 C CNN
+F 4 "1170871" H 7450 4050 60  0001 C CNN "Farnell"
 	1    7450 4050
 	1    0    0    -1
@@
 F 2 "agg:0603" H 8100 3650 50  0001 C CNN
 F 3 "" H 8100 3650 50  0001 C CNN
+F 4 "9330380" H 8100 3650 60  0001 C CNN "Farnell"
 	1    8100 3650
 	1    0    0    -1
 $EndComp
 $Comp
-L 3v3 #PWR405
+L 3v3 #PWR082
 U 1 1 584B9E07
 P 4750 2500
-F 0 "#PWR405" H 4750 2610 50  0001 L CNN
+F 0 "#PWR082" H 4750 2610 50  0001 L CNN
 F 1 "3v3" H 4750 2590 50  0000 C CNN
 F 2 "" H 4750 2500 60  0001 C CNN
@@
 $EndComp
 $Comp
-L 3v3 #PWR418
+L 3v3 #PWR083
 U 1 1 584B9E72
 P 8250 3600
-F 0 "#PWR418" H 8250 3710 50  0001 L CNN
+F 0 "#PWR083" H 8250 3710 50  0001 L CNN
 F 1 "3v3" H 8250 3690 50  0000 C CNN
 F 2 "" H 8250 3600 60  0001 C CNN
@@
 F 2 "agg:0603" H 7500 4450 50  0001 C CNN
 F 3 "" H 7500 4450 50  0001 C CNN
+F 4 "9330399" H 7500 4450 60  0001 C CNN "Farnell"
 	1    7500 4450
 	0    1    1    0
 $EndComp
 $Comp
-L GND #PWR416
+L GND #PWR084
 U 1 1 584BA2FE
 P 7500 4600
-F 0 "#PWR416" H 7370 4640 50  0001 L CNN
+F 0 "#PWR084" H 7370 4640 50  0001 L CNN
 F 1 "GND" H 7500 4500 50  0000 C CNN
 F 2 "" H 7500 4600 60  0001 C CNN
@@
 F 2 "agg:0603" H 5750 4300 50  0001 C CNN
 F 3 "" H 5750 4300 50  0001 C CNN
+F 4 "2627466" H 5750 4300 60  0001 C CNN "Farnell"
 	1    5750 4300
 	-1   0    0    1
@@
 F 2 "agg:0603" H 5750 4100 50  0001 C CNN
 F 3 "" H 5750 4100 50  0001 C CNN
+F 4 "2627466" H 5750 4100 60  0001 C CNN "Farnell"
 	1    5750 4100
 	-1   0    0    1
 $EndComp
 $Comp
-L GND #PWR412
+L GND #PWR085
 U 1 1 584BAE67
 P 5500 4200
-F 0 "#PWR412" H 5370 4240 50  0001 L CNN
+F 0 "#PWR085" H 5370 4240 50  0001 L CNN
 F 1 "GND" H 5500 4100 50  0000 C CNN
 F 2 "" H 5500 4200 60  0001 C CNN
@@
 $EndComp
 $Comp
-L GND #PWR415
+L GND #PWR086
 U 1 1 584BB204
 P 6100 3500
-F 0 "#PWR415" H 5970 3540 50  0001 L CNN
+F 0 "#PWR086" H 5970 3540 50  0001 L CNN
 F 1 "GND" H 6100 3400 50  0000 C CNN
 F 2 "" H 6100 3500 60  0001 C CNN
@@
 F 2 "agg:0603" H 5900 3300 50  0001 C CNN
 F 3 "" H 5900 3300 50  0001 C CNN
+F 4 "1759037" H 5900 3300 60  0001 C CNN "Farnell"
 	1    5900 3300
 	0    -1   -1   0
@@
 F 2 "agg:0603" H 5650 3300 50  0001 C CNN
 F 3 "" H 5650 3300 50  0001 C CNN
+F 4 "2320817" H 5650 3300 60  0001 C CNN "Farnell"
 	1    5650 3300
 	0    -1   -1   0
@@
 F 2 "agg:0603" H 4500 2850 50  0001 C CNN
 F 3 "" H 4500 2850 50  0001 C CNN
+F 4 "2494232" H 4500 2850 60  0001 C CNN "Farnell"
 	1    4500 2850
 	0    -1   -1   0
@@
 F 2 "agg:0603" H 4750 2850 50  0001 C CNN
 F 3 "" H 4750 2850 50  0001 C CNN
+F 4 "1759037" H 4750 2850 60  0001 C CNN "Farnell"
 	1    4750 2850
 	0    -1   -1   0
@@
 $EndComp
 $Comp
-L GND #PWR404
+L GND #PWR087
 U 1 1 584BC166
 P 4500 2900
-F 0 "#PWR404" H 4370 2940 50  0001 L CNN
+F 0 "#PWR087" H 4370 2940 50  0001 L CNN
 F 1 "GND" H 4500 2800 50  0000 C CNN
 F 2 "" H 4500 2900 60  0001 C CNN
@@
 $EndComp
 $Comp
-L GND #PWR414
+L GND #PWR088
 U 1 1 584BC26D
 P 5900 3350
-F 0 "#PWR414" H 5770 3390 50  0001 L CNN
+F 0 "#PWR088" H 5770 3390 50  0001 L CNN
 F 1 "GND" H 5900 3250 50  0000 C CNN
 F 2 "" H 5900 3350 60  0001 C CNN
@@
 $EndComp
 $Comp
-L GND #PWR413
+L GND #PWR089
 U 1 1 584BC2B7
 P 5650 3350
-F 0 "#PWR413" H 5520 3390 50  0001 L CNN
+F 0 "#PWR089" H 5520 3390 50  0001 L CNN
 F 1 "GND" H 5650 3250 50  0000 C CNN
 F 2 "" H 5650 3350 60  0001 C CNN
@@
 $EndComp
 $Comp
-L GND #PWR406
+L GND #PWR090
 U 1 1 584BC475
 P 4750 2900
-F 0 "#PWR406" H 4620 2940 50  0001 L CNN
+F 0 "#PWR090" H 4620 2940 50  0001 L CNN
 F 1 "GND" H 4750 2800 50  0000 C CNN
 F 2 "" H 4750 2900 60  0001 C CNN
@@
 $EndComp
 $Comp
-L PWR #FLG401
+L PWR #FLG091
 U 1 1 584BC5A0
 P 4500 2650
-F 0 "#FLG401" H 4500 2810 50  0001 C CNN
+F 0 "#FLG091" H 4500 2810 50  0001 C CNN
 F 1 "PWR" H 4500 2740 50  0000 C CNN
 F 2 "" H 4500 2650 50  0001 C CNN
@@
 F 2 "agg:0603" H 5100 3100 50  0001 C CNN
 F 3 "" H 5100 3100 50  0001 C CNN
+F 4 "2494232" H 5100 3100 60  0001 C CNN "Farnell"
 	1    5100 3100
 	0    -1   -1   0
@@
 F 2 "agg:0603" H 5350 3100 50  0001 C CNN
 F 3 "" H 5350 3100 50  0001 C CNN
+F 4 "1759037" H 5350 3100 60  0001 C CNN "Farnell"
 	1    5350 3100
 	0    -1   -1   0
 $EndComp
 $Comp
-L GND #PWR410
+L GND #PWR092
 U 1 1 584BCAA1
 P 5100 3150
-F 0 "#PWR410" H 4970 3190 50  0001 L CNN
+F 0 "#PWR092" H 4970 3190 50  0001 L CNN
 F 1 "GND" H 5100 3050 50  0000 C CNN
 F 2 "" H 5100 3150 60  0001 C CNN
@@
 $EndComp
 $Comp
-L GND #PWR411
+L GND #PWR093
 U 1 1 584BCAA8
 P 5350 3150
-F 0 "#PWR411" H 5220 3190 50  0001 L CNN
+F 0 "#PWR093" H 5220 3190 50  0001 L CNN
 F 1 "GND" H 5350 3050 50  0000 C CNN
 F 2 "" H 5350 3150 60  0001 C CNN
@@
 $EndComp
 $Comp
-L 3v3 #PWR409
+L 3v3 #PWR094
 U 1 1 584BCC0A
 P 5050 2900
-F 0 "#PWR409" H 5050 3010 50  0001 L CNN
+F 0 "#PWR094" H 5050 3010 50  0001 L CNN
 F 1 "3v3" H 5050 2990 50  0000 C CNN
 F 2 "" H 5050 2900 60  0001 C CNN
@@
 F 2 "agg:0603" H 4600 3600 50  0001 C CNN
 F 3 "" H 4600 3600 50  0001 C CNN
+F 4 "1759037" H 4600 3600 60  0001 C CNN "Farnell"
 	1    4600 3600
 	1    0    0    -1
@@
 F 2 "agg:0603" H 4600 4000 50  0001 C CNN
 F 3 "" H 4600 4000 50  0001 C CNN
+F 4 "1759037" H 4600 4000 60  0001 C CNN "Farnell"
 	1    4600 4000
 	1    0    0    -1
 $EndComp
 $Comp
-L GND #PWR407
+L GND #PWR095
 U 1 1 584BDBA9
 P 4750 3600
-F 0 "#PWR407" H 4620 3640 50  0001 L CNN
+F 0 "#PWR095" H 4620 3640 50  0001 L CNN
 F 1 "GND" H 4750 3500 50  0000 C CNN
 F 2 "" H 4750 3600 60  0001 C CNN
@@
 $EndComp
 $Comp
-L GND #PWR408
+L GND #PWR096
 U 1 1 584BDCAE
 P 4750 4000
-F 0 "#PWR408" H 4620 4040 50  0001 L CNN
+F 0 "#PWR096" H 4620 4040 50  0001 L CNN
 F 1 "GND" H 4750 3900 50  0000 C CNN
 F 2 "" H 4750 4000 60  0001 C CNN
@@
 CT2
 $Comp
-L GND #PWR417
+L GND #PWR097
 U 1 1 584C02A5
 P 7600 4050
-F 0 "#PWR417" H 7470 4090 50  0001 L CNN
+F 0 "#PWR097" H 7470 4090 50  0001 L CNN
 F 1 "GND" H 7600 3950 50  0000 C CNN
 F 2 "" H 7600 4050 60  0001 C CNN
@@
 F 2 "agg:0603" H 1750 3500 50  0001 C CNN
 F 3 "" H 1750 3500 50  0001 C CNN
+F 4 "9330380" H 1750 3500 60  0001 C CNN "Farnell"
 	1    1750 3500
 	-1   0    0    -1
 $EndComp
 $Comp
-L 3v3 #PWR401
+L 3v3 #PWR098
 U 1 1 584C07D6
 P 1550 3450
-F 0 "#PWR401" H 1550 3560 50  0001 L CNN
+F 0 "#PWR098" H 1550 3560 50  0001 L CNN
 F 1 "3v3" H 1550 3540 50  0000 C CNN
 F 2 "" H 1550 3450 60  0001 C CNN
@@
 $EndComp
 $Comp
-L GND #PWR403
+L GND #PWR099
 U 1 1 584C57B0
 P 2750 5150
-F 0 "#PWR403" H 2620 5190 50  0001 L CNN
+F 0 "#PWR099" H 2620 5190 50  0001 L CNN
 F 1 "GND" H 2750 5050 50  0000 C CNN
 F 2 "" H 2750 5150 60  0001 C CNN
@@
 $EndComp
 $Comp
-L GND #PWR402
+L GND #PWR0100
 U 1 1 584B6EFC
 P 2050 4050
-F 0 "#PWR402" H 1920 4090 50  0001 L CNN
+F 0 "#PWR0100" H 1920 4090 50  0001 L CNN
 F 1 "GND" H 2050 3950 50  0000 C CNN
 F 2 "" H 2050 4050 60  0001 C CNN
@@
 F 2 "agg:0603" H 7450 3350 50  0001 C CNN
 F 3 "" H 7450 3350 50  0001 C CNN
+F 4 "9331050" H 7450 3350 60  0001 C CNN "Farnell"
 	1    7450 3350
 	1    0    0    -1
@@
 F 2 "agg:0603" H 7600 3450 50  0001 C CNN
 F 3 "" H 7600 3450 50  0001 C CNN
+F 4 "9331050" H 7600 3450 60  0001 C CNN "Farnell"
 	1    7600 3450
 	1    0    0    -1
@@
 F 2 "agg:0603" H 7450 3550 50  0001 C CNN
 F 3 "" H 7450 3550 50  0001 C CNN
+F 4 "9331050" H 7450 3550 60  0001 C CNN "Farnell"
 	1    7450 3550
 	1    0    0    -1
