File: hardware/linetime_gps.sch (KiCad schematic (older format))
At the start: 17 parts

Commit message: schematic basically done...
Parts:
- added D301: ESD_DIODE, agg:0402, symbol ESD_DIODE
- L301: renamed from L?; footprint (none) -> agg:0603
- R301: renamed from R?; footprint (none) -> agg:0603
- gave numbers to parts that had none: 15
Connections:
- net GND: now also D301.1
- net at IC303.11 (RF_IN), L301.2, P301.1 (RF): now also D301.2
Other:
- moved on the sheet: P301

Commit message: WIP routing
Parts:
- added C309: 1µ, agg:0603, symbol C
Connections:
- net 3v3: now also C309.1
- net GND: now also C309.2
Changed lines of the file:
@@
 Connection ~ 6950 4000
 $Comp
-L GND #PWR066
+L GND #PWR320
 U 1 1 584A307E
 P 7450 4200
-F 0 "#PWR066" H 7320 4240 50  0001 L CNN
+F 0 "#PWR320" H 7320 4240 50  0001 L CNN
 F 1 "GND" H 7450 4100 50  0000 C CNN
 F 2 "" H 7450 4200 60  0001 C CNN
@@
 $EndComp
 $Comp
-L GND #PWR067
+L GND #PWR319
 U 1 1 584A30E1
 P 7150 3700
-F 0 "#PWR067" H 7020 3740 50  0001 L CNN
+F 0 "#PWR319" H 7020 3740 50  0001 L CNN
 F 1 "GND" H 7150 3600 50  0000 C CNN
 F 2 "" H 7150 3700 60  0001 C CNN
@@
 	6600 3300 6650 3300
 $Comp
-L 3v3 #PWR068
+L 3v3 #PWR317
 U 1 1 584A34A9
 P 5350 2950
-F 0 "#PWR068" H 5350 3060 50  0001 L CNN
+F 0 "#PWR317" H 5350 3060 50  0001 L CNN
 F 1 "3v3" H 5350 3040 50  0000 C CNN
 F 2 "" H 5350 2950 60  0001 C CNN
@@
 $EndComp
 $Comp
-L 3v3 #PWR069
+L 3v3 #PWR312
 U 1 1 584A35BC
 P 5150 3000
-F 0 "#PWR069" H 5150 3110 50  0001 L CNN
+F 0 "#PWR312" H 5150 3110 50  0001 L CNN
 F 1 "3v3" H 5150 3090 50  0000 C CNN
 F 2 "" H 5150 3000 60  0001 C CNN
@@
 	5150 3000 5150 3050
 $Comp
-L GND #PWR070
+L GND #PWR316
 U 1 1 584A35F4
 P 5300 3550
-F 0 "#PWR070" H 5170 3590 50  0001 L CNN
+F 0 "#PWR316" H 5170 3590 50  0001 L CNN
 F 1 "GND" H 5300 3450 50  0000 C CNN
 F 2 "" H 5300 3550 60  0001 C CNN
@@
 Connection ~ 5300 3400
 $Comp
-L GND #PWR071
+L GND #PWR313
 U 1 1 584A366D
 P 5150 3200
-F 0 "#PWR071" H 5020 3240 50  0001 L CNN
+F 0 "#PWR313" H 5020 3240 50  0001 L CNN
 F 1 "GND" H 5150 3100 50  0000 C CNN
 F 2 "" H 5150 3200 60  0001 C CNN
@@
 	4850 5100 5300 5100
 $Comp
-L 3v3 #PWR072
+L 3v3 #PWR314
 U 1 1 584A3402
 P 5250 4750
-F 0 "#PWR072" H 5250 4860 50  0001 L CNN
+F 0 "#PWR314" H 5250 4860 50  0001 L CNN
 F 1 "3v3" H 5250 4840 50  0000 C CNN
 F 2 "" H 5250 4750 60  0001 C CNN
@@
 	5250 4800 5300 4800
 $Comp
-L GND #PWR073
+L GND #PWR315
 U 1 1 584A3457
 P 5250 4900
-F 0 "#PWR073" H 5120 4940 50  0001 L CNN
+F 0 "#PWR315" H 5120 4940 50  0001 L CNN
 F 1 "GND" H 5250 4800 50  0000 C CNN
 F 2 "" H 5250 4900 60  0001 C CNN
@@
 $EndComp
 $Comp
-L 3v3 #PWR074
+L 3v3 #PWR310
 U 1 1 584A34F6
 P 5050 4650
-F 0 "#PWR074" H 5050 4760 50  0001 L CNN
+F 0 "#PWR310" H 5050 4760 50  0001 L CNN
 F 1 "3v3" H 5050 4740 50  0000 C CNN
 F 2 "" H 5050 4650 60  0001 C CNN
@@
 	5050 4650 5050 4700
 $Comp
-L GND #PWR075
+L GND #PWR311
 U 1 1 584A34FD
 P 5050 4850
-F 0 "#PWR075" H 4920 4890 50  0001 L CNN
+F 0 "#PWR311" H 4920 4890 50  0001 L CNN
 F 1 "GND" H 5050 4750 50  0000 C CNN
 F 2 "" H 5050 4850 60  0001 C CNN
@@
 NoConn ~ 6700 4900
 $Comp
-L GND #PWR076
+L GND #PWR318
 U 1 1 584A35BA
 P 6750 5350
-F 0 "#PWR076" H 6620 5390 50  0001 L CNN
+F 0 "#PWR318" H 6620 5390 50  0001 L CNN
 F 1 "GND" H 6750 5250 50  0000 C CNN
 F 2 "" H 6750 5350 60  0001 C CNN
@@
 NoConn ~ 5300 5300
 $Comp
-L GND #PWR077
+L GND #PWR305
 U 1 1 584A37D0
 P 2650 5450
-F 0 "#PWR077" H 2520 5490 50  0001 L CNN
+F 0 "#PWR305" H 2520 5490 50  0001 L CNN
 F 1 "GND" H 2650 5350 50  0000 C CNN
 F 2 "" H 2650 5450 60  0001 C CNN
@@
 $EndComp
 $Comp
-L 3v3 #PWR078
+L 3v3 #PWR301
 U 1 1 584AF153
 P 1100 5250
-F 0 "#PWR078" H 1100 5360 50  0001 L CNN
+F 0 "#PWR301" H 1100 5360 50  0001 L CNN
 F 1 "3v3" H 1100 5340 50  0000 C CNN
 F 2 "" H 1100 5250 60  0001 C CNN
@@
 	1100 5250 1100 5500
 Wire Wire Line
-	1100 5300 1150 5300
+	1000 5300 1150 5300
 Wire Wire Line
 	1100 5400 1150 5400
@@
 Connection ~ 1100 5400
 $Comp
-L GND #PWR079
+L GND #PWR302
 U 1 1 584AF27D
 P 1100 5650
-F 0 "#PWR079" H 970 5690 50  0001 L CNN
+F 0 "#PWR302" H 970 5690 50  0001 L CNN
 F 1 "GND" H 1100 5550 50  0000 C CNN
 F 2 "" H 1100 5650 60  0001 C CNN
@@
 $EndComp
 Wire Wire Line
-	1150 5600 1100 5600
+	1000 5600 1150 5600
 Wire Wire Line
 	1100 5600 1100 5650
@@
 $EndComp
 $Comp
-L GND #PWR080
+L GND #PWR303
 U 1 1 584AF68F
 P 2150 5550
-F 0 "#PWR080" H 2020 5590 50  0001 L CNN
+F 0 "#PWR303" H 2020 5590 50  0001 L CNN
 F 1 "GND" H 2150 5450 50  0000 C CNN
 F 2 "" H 2150 5550 60  0001 C CNN
@@
 $EndComp
 $Comp
-L GND #PWR081
+L GND #PWR304
 U 1 1 584AF6D0
 P 2400 5550
-F 0 "#PWR081" H 2270 5590 50  0001 L CNN
+F 0 "#PWR304" H 2270 5590 50  0001 L CNN
 F 1 "GND" H 2400 5450 50  0000 C CNN
 F 2 "" H 2400 5550 60  0001 C CNN
@@
 	4000 4950 4350 4950
 $Comp
-L GND #PWR082
+L GND #PWR308
 U 1 1 584AFAF5
 P 3700 5450
-F 0 "#PWR082" H 3570 5490 50  0001 L CNN
+F 0 "#PWR308" H 3570 5490 50  0001 L CNN
 F 1 "GND" H 3700 5350 50  0000 C CNN
 F 2 "" H 3700 5450 60  0001 C CNN
@@
 $EndComp
 $Comp
-L 3v3 #PWR083
+L 3v3 #PWR309
 U 1 1 584AFE50
 P 4200 5150
-F 0 "#PWR083" H 4200 5260 50  0001 L CNN
+F 0 "#PWR309" H 4200 5260 50  0001 L CNN
 F 1 "3v3" H 4200 5240 50  0000 C CNN
 F 2 "" H 4200 5150 60  0001 C CNN
@@
 	4200 5200 4200 5150
 $Comp
-L 3v3 #PWR084
+L 3v3 #PWR306
 U 1 1 584B00B4
 P 3500 4750
-F 0 "#PWR084" H 3500 4860 50  0001 L CNN
+F 0 "#PWR306" H 3500 4860 50  0001 L CNN
 F 1 "3v3" H 3500 4840 50  0000 C CNN
 F 2 "" H 3500 4750 60  0001 C CNN
@@
 	3500 4750 3500 4800
 $Comp
-L GND #PWR085
+L GND #PWR307
 U 1 1 584B0154
 P 3500 4950
-F 0 "#PWR085" H 3370 4990 50  0001 L CNN
+F 0 "#PWR307" H 3370 4990 50  0001 L CNN
 F 1 "GND" H 3500 4850 50  0000 C CNN
 F 2 "" H 3500 4950 60  0001 C CNN
@@
 	7450 4100 7450 4200
 Connection ~ 7450 4100
+$Comp
+L C C309
+U 1 1 5853400D
+P 1000 5400
+F 0 "C309" H 1050 5470 50  0000 C CNN
+F 1 "1µ" H 1050 5330 50  0000 C CNN
+F 2 "agg:0603" H 1000 5400 50  0001 C CNN
+F 3 "" H 1000 5400 50  0001 C CNN
+	1    1000 5400
+	0    1    1    0
+$EndComp
+Wire Wire Line
+	1000 5400 1000 5300
+Wire Wire Line
+	1000 5500 1000 5600
+Connection ~ 1100 5600
 $EndSCHEMATC

Commit message: 22 airwires to go
Parts:
- added R1, R2: 10k, agg:0603, symbol R
- added R?: 22, agg:0603, symbol R
Connections:
- net 3v3: now also R1.1, R2.1
- net CS2100_CLK: now also R?.2; no longer IC304.3 (CLK_OUT)
- net CS2100_SCL: now also R2.2
- net CS2100_SDA: now also R1.2
- new net: IC304.3 (CLK_OUT), R?.1
Changed lines of the file:
@@
 EESchema Schematic File Version 2
-LIBS:agg-kicad
 LIBS:linetime-cache
 EELAYER 25 0
@@
 Connection ~ 6950 4000
 $Comp
-L GND #PWR320
+L GND #PWR066
 U 1 1 584A307E
 P 7450 4200
-F 0 "#PWR320" H 7320 4240 50  0001 L CNN
+F 0 "#PWR066" H 7320 4240 50  0001 L CNN
 F 1 "GND" H 7450 4100 50  0000 C CNN
 F 2 "" H 7450 4200 60  0001 C CNN
@@
 $EndComp
 $Comp
-L GND #PWR319
+L GND #PWR067
 U 1 1 584A30E1
 P 7150 3700
-F 0 "#PWR319" H 7020 3740 50  0001 L CNN
+F 0 "#PWR067" H 7020 3740 50  0001 L CNN
 F 1 "GND" H 7150 3600 50  0000 C CNN
 F 2 "" H 7150 3700 60  0001 C CNN
@@
 	6600 3300 6650 3300
 $Comp
-L 3v3 #PWR317
+L 3v3 #PWR068
 U 1 1 584A34A9
 P 5350 2950
-F 0 "#PWR317" H 5350 3060 50  0001 L CNN
+F 0 "#PWR068" H 5350 3060 50  0001 L CNN
 F 1 "3v3" H 5350 3040 50  0000 C CNN
 F 2 "" H 5350 2950 60  0001 C CNN
@@
 $EndComp
 $Comp
-L 3v3 #PWR312
+L 3v3 #PWR069
 U 1 1 584A35BC
 P 5150 3000
-F 0 "#PWR312" H 5150 3110 50  0001 L CNN
+F 0 "#PWR069" H 5150 3110 50  0001 L CNN
 F 1 "3v3" H 5150 3090 50  0000 C CNN
 F 2 "" H 5150 3000 60  0001 C CNN
@@
 	5150 3000 5150 3050
 $Comp
-L GND #PWR316
+L GND #PWR070
 U 1 1 584A35F4
 P 5300 3550
-F 0 "#PWR316" H 5170 3590 50  0001 L CNN
+F 0 "#PWR070" H 5170 3590 50  0001 L CNN
 F 1 "GND" H 5300 3450 50  0000 C CNN
 F 2 "" H 5300 3550 60  0001 C CNN
@@
 Connection ~ 5300 3400
 $Comp
-L GND #PWR313
+L GND #PWR071
 U 1 1 584A366D
 P 5150 3200
-F 0 "#PWR313" H 5020 3240 50  0001 L CNN
+F 0 "#PWR071" H 5020 3240 50  0001 L CNN
 F 1 "GND" H 5150 3100 50  0000 C CNN
 F 2 "" H 5150 3200 60  0001 C CNN
@@
 	4850 5100 5300 5100
 $Comp
-L 3v3 #PWR314
+L 3v3 #PWR072
 U 1 1 584A3402
 P 5250 4750
-F 0 "#PWR314" H 5250 4860 50  0001 L CNN
+F 0 "#PWR072" H 5250 4860 50  0001 L CNN
 F 1 "3v3" H 5250 4840 50  0000 C CNN
 F 2 "" H 5250 4750 60  0001 C CNN
@@
 	5250 4800 5300 4800
 $Comp
-L GND #PWR315
+L GND #PWR073
 U 1 1 584A3457
 P 5250 4900
-F 0 "#PWR315" H 5120 4940 50  0001 L CNN
+F 0 "#PWR073" H 5120 4940 50  0001 L CNN
 F 1 "GND" H 5250 4800 50  0000 C CNN
 F 2 "" H 5250 4900 60  0001 C CNN
@@
 $EndComp
 $Comp
-L 3v3 #PWR310
+L 3v3 #PWR074
 U 1 1 584A34F6
 P 5050 4650
-F 0 "#PWR310" H 5050 4760 50  0001 L CNN
+F 0 "#PWR074" H 5050 4760 50  0001 L CNN
 F 1 "3v3" H 5050 4740 50  0000 C CNN
 F 2 "" H 5050 4650 60  0001 C CNN
@@
 	5050 4650 5050 4700
 $Comp
-L GND #PWR311
+L GND #PWR075
 U 1 1 584A34FD
 P 5050 4850
-F 0 "#PWR311" H 4920 4890 50  0001 L CNN
+F 0 "#PWR075" H 4920 4890 50  0001 L CNN
 F 1 "GND" H 5050 4750 50  0000 C CNN
 F 2 "" H 5050 4850 60  0001 C CNN
@@
 Wire Wire Line
 	5050 4850 5050 4800
-Text HLabel 6800 4800 2    60   Output ~ 0
+Text HLabel 7000 4800 2    60   Output ~ 0
 CS2100_CLK
 Wire Wire Line
@@
 NoConn ~ 6700 4900
 $Comp
-L GND #PWR318
+L GND #PWR076
 U 1 1 584A35BA
 P 6750 5350
-F 0 "#PWR318" H 6620 5390 50  0001 L CNN
+F 0 "#PWR076" H 6620 5390 50  0001 L CNN
 F 1 "GND" H 6750 5250 50  0000 C CNN
 F 2 "" H 6750 5350 60  0001 C CNN
@@
 NoConn ~ 5300 5300
 $Comp
-L GND #PWR305
+L GND #PWR077
 U 1 1 584A37D0
 P 2650 5450
-F 0 "#PWR305" H 2520 5490 50  0001 L CNN
+F 0 "#PWR077" H 2520 5490 50  0001 L CNN
 F 1 "GND" H 2650 5350 50  0000 C CNN
 F 2 "" H 2650 5450 60  0001 C CNN
@@
 $EndComp
 $Comp
-L 3v3 #PWR301
+L 3v3 #PWR078
 U 1 1 584AF153
 P 1100 5250
-F 0 "#PWR301" H 1100 5360 50  0001 L CNN
+F 0 "#PWR078" H 1100 5360 50  0001 L CNN
 F 1 "3v3" H 1100 5340 50  0000 C CNN
 F 2 "" H 1100 5250 60  0001 C CNN
@@
 Connection ~ 1100 5400
 $Comp
-L GND #PWR302
+L GND #PWR079
 U 1 1 584AF27D
 P 1100 5650
-F 0 "#PWR302" H 970 5690 50  0001 L CNN
+F 0 "#PWR079" H 970 5690 50  0001 L CNN
 F 1 "GND" H 1100 5550 50  0000 C CNN
 F 2 "" H 1100 5650 60  0001 C CNN
@@
 $EndComp
 $Comp
-L GND #PWR303
+L GND #PWR080
 U 1 1 584AF68F
 P 2150 5550
-F 0 "#PWR303" H 2020 5590 50  0001 L CNN
+F 0 "#PWR080" H 2020 5590 50  0001 L CNN
 F 1 "GND" H 2150 5450 50  0000 C CNN
 F 2 "" H 2150 5550 60  0001 C CNN
@@
 $EndComp
 $Comp
-L GND #PWR304
+L GND #PWR081
 U 1 1 584AF6D0
 P 2400 5550
-F 0 "#PWR304" H 2270 5590 50  0001 L CNN
+F 0 "#PWR081" H 2270 5590 50  0001 L CNN
 F 1 "GND" H 2400 5450 50  0000 C CNN
 F 2 "" H 2400 5550 60  0001 C CNN
@@
 	4000 4950 4350 4950
 $Comp
-L GND #PWR308
+L GND #PWR082
 U 1 1 584AFAF5
 P 3700 5450
-F 0 "#PWR308" H 3570 5490 50  0001 L CNN
+F 0 "#PWR082" H 3570 5490 50  0001 L CNN
 F 1 "GND" H 3700 5350 50  0000 C CNN
 F 2 "" H 3700 5450 60  0001 C CNN
@@
 $EndComp
 $Comp
-L 3v3 #PWR309
+L 3v3 #PWR083
 U 1 1 584AFE50
 P 4200 5150
-F 0 "#PWR309" H 4200 5260 50  0001 L CNN
+F 0 "#PWR083" H 4200 5260 50  0001 L CNN
 F 1 "3v3" H 4200 5240 50  0000 C CNN
 F 2 "" H 4200 5150 60  0001 C CNN
@@
 	4200 5200 4200 5150
 $Comp
-L 3v3 #PWR306
+L 3v3 #PWR084
 U 1 1 584B00B4
 P 3500 4750
-F 0 "#PWR306" H 3500 4860 50  0001 L CNN
+F 0 "#PWR084" H 3500 4860 50  0001 L CNN
 F 1 "3v3" H 3500 4840 50  0000 C CNN
 F 2 "" H 3500 4750 60  0001 C CNN
@@
 	3500 4750 3500 4800
 $Comp
-L GND #PWR307
+L GND #PWR085
 U 1 1 584B0154
 P 3500 4950
-F 0 "#PWR307" H 3370 4990 50  0001 L CNN
+F 0 "#PWR085" H 3370 4990 50  0001 L CNN
 F 1 "GND" H 3500 4850 50  0000 C CNN
 F 2 "" H 3500 4950 60  0001 C CNN
@@
 	1000 5500 1000 5600
 Connection ~ 1100 5600
+Text HLabel 7400 5800 0    60   BiDi ~ 0
+CS2100_SDA
+Text HLabel 7400 5900 0    60   Output ~ 0
+CS2100_SCL
+$Comp
+L R R1
+U 1 1 585522CD
+P 7450 5600
+F 0 "R1" H 7500 5650 50  0000 C CNN
+F 1 "10k" H 7500 5550 50  0000 C CNN
+F 2 "agg:0603" H 7450 5600 50  0001 C CNN
+F 3 "" H 7450 5600 50  0001 C CNN
+	1    7450 5600
+	0    1    1    0
+$EndComp
+$Comp
+L R R2
+U 1 1 58552749
+P 7650 5600
+F 0 "R2" H 7700 5650 50  0000 C CNN
+F 1 "10k" H 7700 5550 50  0000 C CNN
+F 2 "agg:0603" H 7650 5600 50  0001 C CNN
+F 3 "" H 7650 5600 50  0001 C CNN
+	1    7650 5600
+	0    1    1    0
+$EndComp
+Wire Wire Line
+	7400 5800 7450 5800
+Wire Wire Line
+	7450 5800 7450 5700
+Wire Wire Line
+	7400 5900 7650 5900
+Wire Wire Line
+	7650 5900 7650 5700
+$Comp
+L 3v3 #PWR086
+U 1 1 58552B97
+P 7450 5550
+F 0 "#PWR086" H 7450 5660 50  0001 L CNN
+F 1 "3v3" H 7450 5640 50  0000 C CNN
+F 2 "" H 7450 5550 60  0001 C CNN
+F 3 "" H 7450 5550 60  0001 C CNN
+	1    7450 5550
+	1    0    0    -1
+$EndComp
+Wire Wire Line
+	7450 5550 7450 5600
+$Comp
+L 3v3 #PWR087
+U 1 1 58552C6C
+P 7650 5550
+F 0 "#PWR087" H 7650 5660 50  0001 L CNN
+F 1 "3v3" H 7650 5640 50  0000 C CNN
+F 2 "" H 7650 5550 60  0001 C CNN
+F 3 "" H 7650 5550 60  0001 C CNN
+	1    7650 5550
+	1    0    0    -1
+$EndComp
+Wire Wire Line
+	7650 5550 7650 5600
+$Comp
+L R R?
+U 1 1 585650F7
+P 6800 4800
+F 0 "R?" H 6850 4850 50  0000 C CNN
+F 1 "22" H 6850 4750 50  0000 C CNN
+F 2 "agg:0603" H 6800 4800 50  0001 C CNN
+F 3 "" H 6800 4800 50  0001 C CNN
+	1    6800 4800
+	1    0    0    -1
+$EndComp
+Wire Wire Line
+	7000 4800 6900 4800
 $EndSCHEMATC

Commit message: cleaned up all the fast lines
Parts:
- R303: renamed from R?; value 22 -> 33
Changed lines of the file:
@@
 EESchema Schematic File Version 2
+LIBS:agg-kicad
 LIBS:linetime-cache
 EELAYER 25 0
@@
 Connection ~ 6950 4000
 $Comp
-L GND #PWR066
+L GND #PWR320
 U 1 1 584A307E
 P 7450 4200
-F 0 "#PWR066" H 7320 4240 50  0001 L CNN
+F 0 "#PWR320" H 7320 4240 50  0001 L CNN
 F 1 "GND" H 7450 4100 50  0000 C CNN
 F 2 "" H 7450 4200 60  0001 C CNN
@@
 $EndComp
 $Comp
-L GND #PWR067
+L GND #PWR319
 U 1 1 584A30E1
 P 7150 3700
-F 0 "#PWR067" H 7020 3740 50  0001 L CNN
+F 0 "#PWR319" H 7020 3740 50  0001 L CNN
 F 1 "GND" H 7150 3600 50  0000 C CNN
 F 2 "" H 7150 3700 60  0001 C CNN
@@
 	6600 3300 6650 3300
 $Comp
-L 3v3 #PWR068
+L 3v3 #PWR317
 U 1 1 584A34A9
 P 5350 2950
-F 0 "#PWR068" H 5350 3060 50  0001 L CNN
+F 0 "#PWR317" H 5350 3060 50  0001 L CNN
 F 1 "3v3" H 5350 3040 50  0000 C CNN
 F 2 "" H 5350 2950 60  0001 C CNN
@@
 $EndComp
 $Comp
-L 3v3 #PWR069
+L 3v3 #PWR312
 U 1 1 584A35BC
 P 5150 3000
-F 0 "#PWR069" H 5150 3110 50  0001 L CNN
+F 0 "#PWR312" H 5150 3110 50  0001 L CNN
 F 1 "3v3" H 5150 3090 50  0000 C CNN
 F 2 "" H 5150 3000 60  0001 C CNN
@@
 	5150 3000 5150 3050
 $Comp
-L GND #PWR070
+L GND #PWR316
 U 1 1 584A35F4
 P 5300 3550
-F 0 "#PWR070" H 5170 3590 50  0001 L CNN
+F 0 "#PWR316" H 5170 3590 50  0001 L CNN
 F 1 "GND" H 5300 3450 50  0000 C CNN
 F 2 "" H 5300 3550 60  0001 C CNN
@@
 Connection ~ 5300 3400
 $Comp
-L GND #PWR071
+L GND #PWR313
 U 1 1 584A366D
 P 5150 3200
-F 0 "#PWR071" H 5020 3240 50  0001 L CNN
+F 0 "#PWR313" H 5020 3240 50  0001 L CNN
 F 1 "GND" H 5150 3100 50  0000 C CNN
 F 2 "" H 5150 3200 60  0001 C CNN
@@
 	4850 5100 5300 5100
 $Comp
-L 3v3 #PWR072
+L 3v3 #PWR314
 U 1 1 584A3402
 P 5250 4750
-F 0 "#PWR072" H 5250 4860 50  0001 L CNN
+F 0 "#PWR314" H 5250 4860 50  0001 L CNN
 F 1 "3v3" H 5250 4840 50  0000 C CNN
 F 2 "" H 5250 4750 60  0001 C CNN
@@
 	5250 4800 5300 4800
 $Comp
-L GND #PWR073
+L GND #PWR315
 U 1 1 584A3457
 P 5250 4900
-F 0 "#PWR073" H 5120 4940 50  0001 L CNN
+F 0 "#PWR315" H 5120 4940 50  0001 L CNN
 F 1 "GND" H 5250 4800 50  0000 C CNN
 F 2 "" H 5250 4900 60  0001 C CNN
@@
 $EndComp
 $Comp
-L 3v3 #PWR074
+L 3v3 #PWR310
 U 1 1 584A34F6
 P 5050 4650
-F 0 "#PWR074" H 5050 4760 50  0001 L CNN
+F 0 "#PWR310" H 5050 4760 50  0001 L CNN
 F 1 "3v3" H 5050 4740 50  0000 C CNN
 F 2 "" H 5050 4650 60  0001 C CNN
@@
 	5050 4650 5050 4700
 $Comp
-L GND #PWR075
+L GND #PWR311
 U 1 1 584A34FD
 P 5050 4850
-F 0 "#PWR075" H 4920 4890 50  0001 L CNN
+F 0 "#PWR311" H 4920 4890 50  0001 L CNN
 F 1 "GND" H 5050 4750 50  0000 C CNN
 F 2 "" H 5050 4850 60  0001 C CNN
@@
 NoConn ~ 6700 4900
 $Comp
-L GND #PWR076
+L GND #PWR318
 U 1 1 584A35BA
 P 6750 5350
-F 0 "#PWR076" H 6620 5390 50  0001 L CNN
+F 0 "#PWR318" H 6620 5390 50  0001 L CNN
 F 1 "GND" H 6750 5250 50  0000 C CNN
 F 2 "" H 6750 5350 60  0001 C CNN
@@
 NoConn ~ 5300 5300
 $Comp
-L GND #PWR077
+L GND #PWR305
 U 1 1 584A37D0
 P 2650 5450
-F 0 "#PWR077" H 2520 5490 50  0001 L CNN
+F 0 "#PWR305" H 2520 5490 50  0001 L CNN
 F 1 "GND" H 2650 5350 50  0000 C CNN
 F 2 "" H 2650 5450 60  0001 C CNN
@@
 $EndComp
 $Comp
-L 3v3 #PWR078
+L 3v3 #PWR301
 U 1 1 584AF153
 P 1100 5250
-F 0 "#PWR078" H 1100 5360 50  0001 L CNN
+F 0 "#PWR301" H 1100 5360 50  0001 L CNN
 F 1 "3v3" H 1100 5340 50  0000 C CNN
 F 2 "" H 1100 5250 60  0001 C CNN
@@
 Connection ~ 1100 5400
 $Comp
-L GND #PWR079
+L GND #PWR302
 U 1 1 584AF27D
 P 1100 5650
-F 0 "#PWR079" H 970 5690 50  0001 L CNN
+F 0 "#PWR302" H 970 5690 50  0001 L CNN
 F 1 "GND" H 1100 5550 50  0000 C CNN
 F 2 "" H 1100 5650 60  0001 C CNN
@@
 $EndComp
 $Comp
-L GND #PWR080
+L GND #PWR303
 U 1 1 584AF68F
 P 2150 5550
-F 0 "#PWR080" H 2020 5590 50  0001 L CNN
+F 0 "#PWR303" H 2020 5590 50  0001 L CNN
 F 1 "GND" H 2150 5450 50  0000 C CNN
 F 2 "" H 2150 5550 60  0001 C CNN
@@
 $EndComp
 $Comp
-L GND #PWR081
+L GND #PWR304
 U 1 1 584AF6D0
 P 2400 5550
-F 0 "#PWR081" H 2270 5590 50  0001 L CNN
+F 0 "#PWR304" H 2270 5590 50  0001 L CNN
 F 1 "GND" H 2400 5450 50  0000 C CNN
 F 2 "" H 2400 5550 60  0001 C CNN
@@
 	4000 4950 4350 4950
 $Comp
-L GND #PWR082
+L GND #PWR308
 U 1 1 584AFAF5
 P 3700 5450
-F 0 "#PWR082" H 3570 5490 50  0001 L CNN
+F 0 "#PWR308" H 3570 5490 50  0001 L CNN
 F 1 "GND" H 3700 5350 50  0000 C CNN
 F 2 "" H 3700 5450 60  0001 C CNN
@@
 $EndComp
 $Comp
-L 3v3 #PWR083
+L 3v3 #PWR309
 U 1 1 584AFE50
 P 4200 5150
-F 0 "#PWR083" H 4200 5260 50  0001 L CNN
+F 0 "#PWR309" H 4200 5260 50  0001 L CNN
 F 1 "3v3" H 4200 5240 50  0000 C CNN
 F 2 "" H 4200 5150 60  0001 C CNN
@@
 	4200 5200 4200 5150
 $Comp
-L 3v3 #PWR084
+L 3v3 #PWR306
 U 1 1 584B00B4
 P 3500 4750
-F 0 "#PWR084" H 3500 4860 50  0001 L CNN
+F 0 "#PWR306" H 3500 4860 50  0001 L CNN
 F 1 "3v3" H 3500 4840 50  0000 C CNN
 F 2 "" H 3500 4750 60  0001 C CNN
@@
 	3500 4750 3500 4800
 $Comp
-L GND #PWR085
+L GND #PWR307
 U 1 1 584B0154
 P 3500 4950
-F 0 "#PWR085" H 3370 4990 50  0001 L CNN
+F 0 "#PWR307" H 3370 4990 50  0001 L CNN
 F 1 "GND" H 3500 4850 50  0000 C CNN
 F 2 "" H 3500 4950 60  0001 C CNN
@@
 	7650 5900 7650 5700
 $Comp
-L 3v3 #PWR086
+L 3v3 #PWR321
 U 1 1 58552B97
 P 7450 5550
-F 0 "#PWR086" H 7450 5660 50  0001 L CNN
+F 0 "#PWR321" H 7450 5660 50  0001 L CNN
 F 1 "3v3" H 7450 5640 50  0000 C CNN
 F 2 "" H 7450 5550 60  0001 C CNN
@@
 	7450 5550 7450 5600
 $Comp
-L 3v3 #PWR087
+L 3v3 #PWR322
 U 1 1 58552C6C
 P 7650 5550
-F 0 "#PWR087" H 7650 5660 50  0001 L CNN
+F 0 "#PWR322" H 7650 5660 50  0001 L CNN
 F 1 "3v3" H 7650 5640 50  0000 C CNN
 F 2 "" H 7650 5550 60  0001 C CNN
@@
 	7650 5550 7650 5600
 $Comp
-L R R?
+L R R303
 U 1 1 585650F7
 P 6800 4800
-F 0 "R?" H 6850 4850 50  0000 C CNN
-F 1 "22" H 6850 4750 50  0000 C CNN
+F 0 "R303" H 6850 4850 50  0000 C CNN
+F 1 "33" H 6850 4750 50  0000 C CNN
 F 2 "agg:0603" H 6800 4800 50  0001 C CNN
 F 3 "" H 6800 4800 50  0001 C CNN
