File: hardware/linetime_gps.sch (KiCad schematic (older format))
At the start: 22 parts, among them IC301 ADP3335, IC302 NC7SZ04, IC303 MAX-M8Q, IC304 CS2100-CP, P301 COAX, Y301 26M TCXO

Commit message: add farnell part numbers for passives
Parts:
- C301, C308: Farnell (none) -> 1759102
- C302, C309: Farnell (none) -> 1759407
- C303, C305, C306, C307: Farnell (none) -> 1759037
- C304: Farnell (none) -> 1759135
- L301: Farnell (none) -> 2424723
- R1, R2: Farnell (none) -> 9330399
- R301: Farnell (none) -> 9330410
- R302: Farnell (none) -> 9330429
- R303: Farnell (none) -> 9331050
Changed lines of the file:
@@
 F 2 "agg:0603" H 6700 3800 50  0001 C CNN
 F 3 "" H 6700 3800 50  0001 C CNN
+F 4 "9330429" H 6700 3800 60  0001 C CNN "Farnell"
 	1    6700 3800
 	1    0    0    -1
@@
 F 2 "agg:0603" H 6950 3850 50  0001 C CNN
 F 3 "" H 6950 3850 50  0001 C CNN
+F 4 "2424723" H 6950 3850 60  0001 C CNN "Farnell"
 	1    6950 3850
 	0    1    1    0
@@
 Connection ~ 6950 4000
 $Comp
-L GND #PWR320
+L GND #PWR060
 U 1 1 584A307E
 P 7450 4200
-F 0 "#PWR320" H 7320 4240 50  0001 L CNN
+F 0 "#PWR060" H 7320 4240 50  0001 L CNN
 F 1 "GND" H 7450 4100 50  0000 C CNN
 F 2 "" H 7450 4200 60  0001 C CNN
@@
 F 2 "agg:0603" H 7000 3700 50  0001 C CNN
 F 3 "" H 7000 3700 50  0001 C CNN
+F 4 "1759102" H 7000 3700 60  0001 C CNN "Farnell"
 	1    7000 3700
 	1    0    0    -1
 $EndComp
 $Comp
-L GND #PWR319
+L GND #PWR061
 U 1 1 584A30E1
 P 7150 3700
-F 0 "#PWR319" H 7020 3740 50  0001 L CNN
+F 0 "#PWR061" H 7020 3740 50  0001 L CNN
 F 1 "GND" H 7150 3600 50  0000 C CNN
 F 2 "" H 7150 3700 60  0001 C CNN
@@
 	6600 3300 6650 3300
 $Comp
-L 3v3 #PWR317
+L 3v3 #PWR062
 U 1 1 584A34A9
 P 5350 2950
-F 0 "#PWR317" H 5350 3060 50  0001 L CNN
+F 0 "#PWR062" H 5350 3060 50  0001 L CNN
 F 1 "3v3" H 5350 3040 50  0000 C CNN
 F 2 "" H 5350 2950 60  0001 C CNN
@@
 F 2 "agg:0603" H 5150 3050 50  0001 C CNN
 F 3 "" H 5150 3050 50  0001 C CNN
+F 4 "1759037" H 5150 3050 60  0001 C CNN "Farnell"
 	1    5150 3050
 	0    1    1    0
 $EndComp
 $Comp
-L 3v3 #PWR312
+L 3v3 #PWR063
 U 1 1 584A35BC
 P 5150 3000
-F 0 "#PWR312" H 5150 3110 50  0001 L CNN
+F 0 "#PWR063" H 5150 3110 50  0001 L CNN
 F 1 "3v3" H 5150 3090 50  0000 C CNN
 F 2 "" H 5150 3000 60  0001 C CNN
@@
 	5150 3000 5150 3050
 $Comp
-L GND #PWR316
+L GND #PWR064
 U 1 1 584A35F4
 P 5300 3550
-F 0 "#PWR316" H 5170 3590 50  0001 L CNN
+F 0 "#PWR064" H 5170 3590 50  0001 L CNN
 F 1 "GND" H 5300 3450 50  0000 C CNN
 F 2 "" H 5300 3550 60  0001 C CNN
@@
 Connection ~ 5300 3400
 $Comp
-L GND #PWR313
+L GND #PWR065
 U 1 1 584A366D
 P 5150 3200
-F 0 "#PWR313" H 5020 3240 50  0001 L CNN
+F 0 "#PWR065" H 5020 3240 50  0001 L CNN
 F 1 "GND" H 5150 3100 50  0000 C CNN
 F 2 "" H 5150 3200 60  0001 C CNN
@@
 	4850 5100 5300 5100
 $Comp
-L 3v3 #PWR314
+L 3v3 #PWR066
 U 1 1 584A3402
 P 5250 4750
-F 0 "#PWR314" H 5250 4860 50  0001 L CNN
+F 0 "#PWR066" H 5250 4860 50  0001 L CNN
 F 1 "3v3" H 5250 4840 50  0000 C CNN
 F 2 "" H 5250 4750 60  0001 C CNN
@@
 	5250 4800 5300 4800
 $Comp
-L GND #PWR315
+L GND #PWR067
 U 1 1 584A3457
 P 5250 4900
-F 0 "#PWR315" H 5120 4940 50  0001 L CNN
+F 0 "#PWR067" H 5120 4940 50  0001 L CNN
 F 1 "GND" H 5250 4800 50  0000 C CNN
 F 2 "" H 5250 4900 60  0001 C CNN
@@
 F 2 "agg:0603" H 5050 4700 50  0001 C CNN
 F 3 "" H 5050 4700 50  0001 C CNN
+F 4 "1759037" H 5050 4700 60  0001 C CNN "Farnell"
 	1    5050 4700
 	0    1    1    0
 $EndComp
 $Comp
-L 3v3 #PWR310
+L 3v3 #PWR068
 U 1 1 584A34F6
 P 5050 4650
-F 0 "#PWR310" H 5050 4760 50  0001 L CNN
+F 0 "#PWR068" H 5050 4760 50  0001 L CNN
 F 1 "3v3" H 5050 4740 50  0000 C CNN
 F 2 "" H 5050 4650 60  0001 C CNN
@@
 	5050 4650 5050 4700
 $Comp
-L GND #PWR311
+L GND #PWR069
 U 1 1 584A34FD
 P 5050 4850
-F 0 "#PWR311" H 4920 4890 50  0001 L CNN
+F 0 "#PWR069" H 4920 4890 50  0001 L CNN
 F 1 "GND" H 5050 4750 50  0000 C CNN
 F 2 "" H 5050 4850 60  0001 C CNN
@@
 NoConn ~ 6700 4900
 $Comp
-L GND #PWR318
+L GND #PWR070
 U 1 1 584A35BA
 P 6750 5350
-F 0 "#PWR318" H 6620 5390 50  0001 L CNN
+F 0 "#PWR070" H 6620 5390 50  0001 L CNN
 F 1 "GND" H 6750 5250 50  0000 C CNN
 F 2 "" H 6750 5350 60  0001 C CNN
@@
 NoConn ~ 5300 5300
 $Comp
-L GND #PWR305
+L GND #PWR071
 U 1 1 584A37D0
 P 2650 5450
-F 0 "#PWR305" H 2520 5490 50  0001 L CNN
+F 0 "#PWR071" H 2520 5490 50  0001 L CNN
 F 1 "GND" H 2650 5350 50  0000 C CNN
 F 2 "" H 2650 5450 60  0001 C CNN
@@
 F 2 "agg:0603" H 3450 5300 50  0001 C CNN
 F 3 "" H 3450 5300 50  0001 C CNN
+F 4 "1759135" H 3450 5300 60  0001 C CNN "Farnell"
 	1    3450 5300
 	1    0    0    -1
@@
 $EndComp
 $Comp
-L 3v3 #PWR301
+L 3v3 #PWR072
 U 1 1 584AF153
 P 1100 5250
-F 0 "#PWR301" H 1100 5360 50  0001 L CNN
+F 0 "#PWR072" H 1100 5360 50  0001 L CNN
 F 1 "3v3" H 1100 5340 50  0000 C CNN
 F 2 "" H 1100 5250 60  0001 C CNN
@@
 Connection ~ 1100 5400
 $Comp
-L GND #PWR302
+L GND #PWR073
 U 1 1 584AF27D
 P 1100 5650
-F 0 "#PWR302" H 970 5690 50  0001 L CNN
+F 0 "#PWR073" H 970 5690 50  0001 L CNN
 F 1 "GND" H 1100 5550 50  0000 C CNN
 F 2 "" H 1100 5650 60  0001 C CNN
@@
 F 2 "agg:0603" H 1850 5600 50  0001 C CNN
 F 3 "" H 1850 5600 50  0001 C CNN
+F 4 "1759102" H 1850 5600 60  0001 C CNN "Farnell"
 	1    1850 5600
 	1    0    0    -1
@@
 F 2 "agg:0603" H 2150 5400 50  0001 C CNN
 F 3 "" H 2150 5400 50  0001 C CNN
+F 4 "1759407" H 2150 5400 60  0001 C CNN "Farnell"
 	1    2150 5400
 	0    1    1    0
@@
 F 2 "agg:0603" H 2400 5400 50  0001 C CNN
 F 3 "" H 2400 5400 50  0001 C CNN
+F 4 "1759037" H 2400 5400 60  0001 C CNN "Farnell"
 	1    2400 5400
 	0    1    1    0
 $EndComp
 $Comp
-L GND #PWR303
+L GND #PWR074
 U 1 1 584AF68F
 P 2150 5550
-F 0 "#PWR303" H 2020 5590 50  0001 L CNN
+F 0 "#PWR074" H 2020 5590 50  0001 L CNN
 F 1 "GND" H 2150 5450 50  0000 C CNN
 F 2 "" H 2150 5550 60  0001 C CNN
@@
 $EndComp
 $Comp
-L GND #PWR304
+L GND #PWR075
 U 1 1 584AF6D0
 P 2400 5550
-F 0 "#PWR304" H 2270 5590 50  0001 L CNN
+F 0 "#PWR075" H 2270 5590 50  0001 L CNN
 F 1 "GND" H 2400 5450 50  0000 C CNN
 F 2 "" H 2400 5550 60  0001 C CNN
@@
 F 2 "agg:0603" H 3900 4950 50  0001 C CNN
 F 3 "" H 3900 4950 50  0001 C CNN
+F 4 "9330410" H 3900 4950 60  0001 C CNN "Farnell"
 	1    3900 4950
 	1    0    0    -1
@@
 	4000 4950 4350 4950
 $Comp
-L GND #PWR308
+L GND #PWR076
 U 1 1 584AFAF5
 P 3700 5450
-F 0 "#PWR308" H 3570 5490 50  0001 L CNN
+F 0 "#PWR076" H 3570 5490 50  0001 L CNN
 F 1 "GND" H 3700 5350 50  0000 C CNN
 F 2 "" H 3700 5450 60  0001 C CNN
@@
 F 2 "agg:0603" H 3500 4800 50  0001 C CNN
 F 3 "" H 3500 4800 50  0001 C CNN
+F 4 "1759037" H 3500 4800 60  0001 C CNN "Farnell"
 	1    3500 4800
 	0    1    1    0
 $EndComp
 $Comp
-L 3v3 #PWR309
+L 3v3 #PWR077
 U 1 1 584AFE50
 P 4200 5150
-F 0 "#PWR309" H 4200 5260 50  0001 L CNN
+F 0 "#PWR077" H 4200 5260 50  0001 L CNN
 F 1 "3v3" H 4200 5240 50  0000 C CNN
 F 2 "" H 4200 5150 60  0001 C CNN
@@
 	4200 5200 4200 5150
 $Comp
-L 3v3 #PWR306
+L 3v3 #PWR078
 U 1 1 584B00B4
 P 3500 4750
-F 0 "#PWR306" H 3500 4860 50  0001 L CNN
+F 0 "#PWR078" H 3500 4860 50  0001 L CNN
 F 1 "3v3" H 3500 4840 50  0000 C CNN
 F 2 "" H 3500 4750 60  0001 C CNN
@@
 	3500 4750 3500 4800
 $Comp
-L GND #PWR307
+L GND #PWR079
 U 1 1 584B0154
 P 3500 4950
-F 0 "#PWR307" H 3370 4990 50  0001 L CNN
+F 0 "#PWR079" H 3370 4990 50  0001 L CNN
 F 1 "GND" H 3500 4850 50  0000 C CNN
 F 2 "" H 3500 4950 60  0001 C CNN
@@
 F 2 "agg:0603" H 1000 5400 50  0001 C CNN
 F 3 "" H 1000 5400 50  0001 C CNN
+F 4 "1759407" H 1000 5400 60  0001 C CNN "Farnell"
 	1    1000 5400
 	0    1    1    0
@@
 F 2 "agg:0603" H 7450 5600 50  0001 C CNN
 F 3 "" H 7450 5600 50  0001 C CNN
+F 4 "9330399" H 7450 5600 60  0001 C CNN "Farnell"
 	1    7450 5600
 	0    1    1    0
@@
 F 2 "agg:0603" H 7650 5600 50  0001 C CNN
 F 3 "" H 7650 5600 50  0001 C CNN
+F 4 "9330399" H 7650 5600 60  0001 C CNN "Farnell"
 	1    7650 5600
 	0    1    1    0
@@
 	7650 5900 7650 5700
 $Comp
-L 3v3 #PWR321
+L 3v3 #PWR080
 U 1 1 58552B97
 P 7450 5550
-F 0 "#PWR321" H 7450 5660 50  0001 L CNN
+F 0 "#PWR080" H 7450 5660 50  0001 L CNN
 F 1 "3v3" H 7450 5640 50  0000 C CNN
 F 2 "" H 7450 5550 60  0001 C CNN
@@
 	7450 5550 7450 5600
 $Comp
-L 3v3 #PWR322
+L 3v3 #PWR081
 U 1 1 58552C6C
 P 7650 5550
-F 0 "#PWR322" H 7650 5660 50  0001 L CNN
+F 0 "#PWR081" H 7650 5660 50  0001 L CNN
 F 1 "3v3" H 7650 5640 50  0000 C CNN
 F 2 "" H 7650 5550 60  0001 C CNN
@@
 F 2 "agg:0603" H 6800 4800 50  0001 C CNN
 F 3 "" H 6800 4800 50  0001 C CNN
+F 4 "9331050" H 6800 4800 60  0001 C CNN "Farnell"
 	1    6800 4800
 	1    0    0    -1
