File: hardware/linetime_mains.sch (KiCad schematic (older format))
At the start: 25 parts, among them IC201 VTX-214-003-105, IC202 ADCMP601, IC203 ADA4528-2, J201 FUSED INLET, T201 AVB0.35/2/6, X201 FUSEHOLDER

Commit message: schematic basically done...
Parts:
- C201, C202: footprint (none) -> agg:B32921; Farnell 1609517 -> 2395807
- C203: footprint (none) -> agg:B32921; Farnell 1673308 -> 2112770
- L201: value L -> FB; footprint (none) -> agg:0603; Farnell (none) -> 1669708
- R203, R204: footprint (none) -> agg:0603
- gave numbers to parts that had none: 4
- renumbered C204 to C207, C205 to C208, C207 to C209, C206 to C210, C208 to C211, C209 to C212, IC202 to IC203, IC203 to IC204
Connections:
- net MAINS_5V: no longer C204.1, IC202.6 (SD), IC202.7 (IN), IC202.8 (IN)
- net MAINS renamed MAINS_WAVE
- new net VCC: C204.1, IC202.6 (SD), IC202.7 (IN), IC202.8 (IN)
Other:
- moved on the sheet: C204, C205, C206, IC202

Commit message: WIP routing
Parts:
- added R205: 22, agg:0603, symbol R
- C209: value 100n -> 10n
Connections:
- net MAINS_BIAS: now also T201.7; no longer T201.5
- net MAINS_ZC: now also R205.2; no longer IC203.1 (Q)
- net at C207.1, L202.1: now also T201.8; no longer T201.6
- new net: IC203.1 (Q), R205.1
Other:
- moved on the sheet: C201, C202, C203, IC201, J201, L201, T201, X201

Commit message: cleaned up all the fast lines
Parts:
- removed L202: ~, agg:0603, symbol L
- added R206: 100, agg:0603, symbol R
- C207: value ~ -> 1n
- R205: value 22 -> 33
Connections:
- net at T201.8: now also R206.2; no longer C207.1
- net at R201.2: now also C207.1, R206.1
Other:
- moved on the sheet: C207, C208, R201

Commit message: add farnell part numbers for passives
Parts:
- C204, C206: Farnell (none) -> 1759407
- C205, C209, C212: Farnell (none) -> 1759102
- C207: Farnell (none) -> 2627458
- C208, C210, C211: Farnell (none) -> 1759037
- R203: Farnell (none) -> 2447743
- R205: Farnell (none) -> 9331050
- R206: Farnell (none) -> 9330364
