File: hardware/linetime_ui.sch (KiCad schematic (older format))
At the start: 0 parts

Commit message: schematic basically done...
Parts:
- added C601, C605, C608: 10µ, agg:0603, symbol C
- added C602, C603, C607, C609: 100n, agg:0603, symbol C
- added C604, C606: 47n, agg:0603, symbol C
- added C610, C611: 10n, agg:0603, symbol C
- added D601, D602, D603, D604: ~, agg:SOD-123, symbol D
- added D605, D606, D607, D608: ESD_DIODE, agg:0402, symbol ESD_DIODE
- added IC601: ER-TFT023-1, agg:ER-CON50HT-1, symbol ER-TFT024-3
- added IC602: SSM2305, agg:MSOP-8, symbol SSM2305
- added IC603: AR1021, agg:SSOP-20, symbol AR1021
- added LS601: KSSG1708, agg:KSSG1708, symbol SOUNDER
- added Q601: NFET, agg:SOT-23, symbol NFET
- added R601, R602: 1k, agg:0603, symbol R
- added R603, R604: 110k, agg:0603, symbol R
- added R605: 20k, agg:0603, symbol R
- added R606: 10k, agg:0603, symbol R
Connections:
- new net: IC602.5 (OUT+), LS601.1
- new net: IC602.8 (OUT-), LS601.2
- new net: IC602.3 (IN+), R604.2
- new net: IC602.4 (IN-), R603.2
- new net: D601.1, D602.1, D603.1, D604.1, Q601.3 (D)
- new net: D603.2, IC601.2 (LEDK1)
- new net: C604.2, R603.1
- new net: D601.2, IC601.3 (LEDK2)
- new net: D604.2, IC601.4 (LEDK3)
- new net: D602.2, IC601.5 (LEDK4)
- new net: IC603.5 (WAKE), R605.2
- new net: C606.2, R604.1
- new net: IC601.34 (SDI), R602.1
- new net: Q601.1 (G), R601.1
- new net 3v3: C601.1, C602.1, C603.1, C608.1, C609.1, IC601.1 (LEDA), IC601.35 (RD), IC601.40 (VDDI), IC601.41 (VDDI), IC601.42 (VCI), IC601.6 (IM0), IC601.7 (IM1), IC601.8 (IM2), IC601.9 (IM3), IC603.1 (VDD), IC603.2 (M1)
- new net B2: IC601.32 (DB0)
- new net B3: IC601.31 (DB1)
- new net B4: IC601.30 (DB2)
- new net B5: IC601.29 (DB3)
- new net B6: IC601.28 (DB4)
- new net B7: IC601.27 (DB5)
- new net BACKLIGHT: R601.2
- new net DE: IC601.14 (DE)
- new net DOTCLK: IC601.13 (DOTCLK)
- new net G2: IC601.26 (DB6)
- new net G3: IC601.25 (DB7)
- new net G4: IC601.24 (DB8)
- new net G5: IC601.23 (DB9)
- new net G6: IC601.22 (DB10)
- new net G7: IC601.21 (DB11)
- new net GND: C601.2, C602.2, C603.2, C604.1, C605.2, C607.2, C608.2, C609.2, C610.2, C611.2, D605.2, D606.2, D607.2, D608.2, IC601.43 (GND), IC601.48 (GND), IC601.49 (GND), IC601.50 (GND), IC602.7 (GND), IC603.14 (SX+), IC603.17 (5WSX-), IC603.20 (VSS), IC603.3 (SY-), IC603.4 (M2), IC603.7 (SY+), Q601.2 (S)
- new net HSYNC: IC601.12 (HSYNC)
- new net R2: IC601.20 (DB12)
- new net R3: IC601.19 (DB13)
- new net R4: IC601.18 (DB14)
- new net R5: IC601.17 (DB15)
- new net R6: IC601.16 (DB16)
- new net R7: IC601.15 (DB17)
- new net SOUNDER: C606.1
- new net SOUNDER_~SD: IC602.1 (~SD), R606.2
- new net TFT_DCX: IC601.36 (WRX)
- new net TFT_RESET: IC601.10 (RESET)
- new net TFT_SCL: IC601.37 (D/CX)
- new net TFT_SDA: R602.2
- new net TFT_~CS: IC601.38 (CSX)
- new net TOUCH_INT: IC603.6 (SIQ)
- new net TOUCH_SCK: IC603.11 (SCK/SCL)
- new net TOUCH_SDI: IC603.13 (SDI/SDA)
- new net TOUCH_SDO: IC603.9 (SDO)
- new net TOUCH_~CS: IC603.8 (SS)
- new net VCC: C605.1, C607.1, IC602.6 (VDD), R606.1
- new net VSYNC: IC601.11 (VSYNC)
- new net X+: C610.1, D608.1, IC601.44 (X+), IC603.18 (X+)
- new net X-: D606.1, IC601.46 (X-), IC603.19 (X-), R605.1
- new net Y+: D607.1, IC601.45 (Y+), IC603.15 (Y+)
- new net Y-: C611.1, D605.1, IC601.47 (Y-), IC603.16 (Y-)
- no-connect marks 0 -> 2
Other:
- note added: "LCD SCREEN"
- note added: "LOUDSPEAKER"
- note added: "TOUCHSCREEN CONTROLLER"

Commit message: WIP routing
Connections:
- net 3v3: no longer IC601.1 (LEDA)
- net VCC: now also IC601.1 (LEDA)
Changed lines of the file:
@@
 $EndComp
 $Comp
-L GND #PWR0114
+L GND #PWR607
 U 1 1 58516C23
 P 4000 2350
-F 0 "#PWR0114" H 3870 2390 50  0001 L CNN
+F 0 "#PWR607" H 3870 2390 50  0001 L CNN
 F 1 "GND" H 4000 2250 50  0000 C CNN
 F 2 "" H 4000 2350 60  0001 C CNN
@@
 $EndComp
 $Comp
-L GND #PWR0115
+L GND #PWR604
 U 1 1 58516C74
 P 3750 2350
-F 0 "#PWR0115" H 3620 2390 50  0001 L CNN
+F 0 "#PWR604" H 3620 2390 50  0001 L CNN
 F 1 "GND" H 3750 2250 50  0000 C CNN
 F 2 "" H 3750 2350 60  0001 C CNN
@@
 $EndComp
 $Comp
-L GND #PWR0116
+L GND #PWR602
 U 1 1 58516C8E
 P 3500 2350
-F 0 "#PWR0116" H 3370 2390 50  0001 L CNN
+F 0 "#PWR602" H 3370 2390 50  0001 L CNN
 F 1 "GND" H 3500 2250 50  0000 C CNN
 F 2 "" H 3500 2350 60  0001 C CNN
@@
 $EndComp
 $Comp
-L 3v3 #PWR0117
+L 3v3 #PWR609
 U 1 1 585171C0
 P 4250 2150
-F 0 "#PWR0117" H 4250 2260 50  0001 L CNN
+F 0 "#PWR609" H 4250 2260 50  0001 L CNN
 F 1 "3v3" H 4250 2240 50  0000 C CNN
 F 2 "" H 4250 2150 60  0001 C CNN
@@
 $EndComp
 $Comp
-L 3v3 #PWR0118
+L 3v3 #PWR606
 U 1 1 58517291
 P 4000 2150
-F 0 "#PWR0118" H 4000 2260 50  0001 L CNN
+F 0 "#PWR606" H 4000 2260 50  0001 L CNN
 F 1 "3v3" H 4000 2240 50  0000 C CNN
 F 2 "" H 4000 2150 60  0001 C CNN
@@
 $EndComp
 $Comp
-L 3v3 #PWR0119
+L 3v3 #PWR603
 U 1 1 585172AB
 P 3750 2150
-F 0 "#PWR0119" H 3750 2260 50  0001 L CNN
+F 0 "#PWR603" H 3750 2260 50  0001 L CNN
 F 1 "3v3" H 3750 2240 50  0000 C CNN
 F 2 "" H 3750 2150 60  0001 C CNN
@@
 $EndComp
 $Comp
-L 3v3 #PWR0120
+L 3v3 #PWR601
 U 1 1 585172C5
 P 3500 2150
-F 0 "#PWR0120" H 3500 2260 50  0001 L CNN
+F 0 "#PWR601" H 3500 2260 50  0001 L CNN
 F 1 "3v3" H 3500 2240 50  0000 C CNN
 F 2 "" H 3500 2150 60  0001 C CNN
@@
 $EndComp
 $Comp
-L GND #PWR0121
+L GND #PWR610
 U 1 1 58517460
 P 4250 2950
-F 0 "#PWR0121" H 4120 2990 50  0001 L CNN
+F 0 "#PWR610" H 4120 2990 50  0001 L CNN
 F 1 "GND" H 4250 2850 50  0000 C CNN
 F 2 "" H 4250 2950 60  0001 C CNN
@@
 $EndComp
 $Comp
-L 3v3 #PWR0122
+L 3v3 #PWR611
 U 1 1 58517599
 P 4250 3650
-F 0 "#PWR0122" H 4250 3760 50  0001 L CNN
+F 0 "#PWR611" H 4250 3760 50  0001 L CNN
 F 1 "3v3" H 4250 3740 50  0000 C CNN
 F 2 "" H 4250 3650 60  0001 C CNN
@@
 $EndComp
 $Comp
-L 3v3 #PWR0123
+L 3v3 #PWR612
 U 1 1 58517717
 P 4250 5000
-F 0 "#PWR0123" H 4250 5110 50  0001 L CNN
+F 0 "#PWR612" H 4250 5110 50  0001 L CNN
 F 1 "3v3" H 4250 5090 50  0000 C CNN
 F 2 "" H 4250 5000 60  0001 C CNN
@@
 	1    4250 5000
 	0    -1   -1   0
-$EndComp
-$Comp
-L 3v3 #PWR0124
-U 1 1 58517BDD
-P 4100 3050
-F 0 "#PWR0124" H 4100 3160 50  0001 L CNN
-F 1 "3v3" H 4100 3140 50  0000 C CNN
-F 2 "" H 4100 3050 60  0001 C CNN
-F 3 "" H 4100 3050 60  0001 C CNN
-	1    4100 3050
-	1    0    0    -1
 $EndComp
 $Comp
@@
 $EndComp
 $Comp
-L GND #PWR0125
+L GND #PWR605
 U 1 1 58518B57
 P 3900 3950
-F 0 "#PWR0125" H 3770 3990 50  0001 L CNN
+F 0 "#PWR605" H 3770 3990 50  0001 L CNN
 F 1 "GND" H 3900 3850 50  0000 C CNN
 F 2 "" H 3900 3950 60  0001 C CNN
@@
 $EndComp
 $Comp
-L VCC #PWR0126
+L VCC #PWR624
 U 1 1 5850D743
 P 8100 2500
-F 0 "#PWR0126" H 8100 2610 50  0001 L CNN
+F 0 "#PWR624" H 8100 2610 50  0001 L CNN
 F 1 "VCC" H 8100 2590 50  0000 C CNN
 F 2 "" H 8100 2500 60  0001 C CNN
@@
 $EndComp
 $Comp
-L GND #PWR0127
+L GND #PWR625
 U 1 1 5850D7F7
 P 8100 2700
-F 0 "#PWR0127" H 7970 2740 50  0001 L CNN
+F 0 "#PWR625" H 7970 2740 50  0001 L CNN
 F 1 "GND" H 8100 2600 50  0000 C CNN
 F 2 "" H 8100 2700 60  0001 C CNN
@@
 $EndComp
 $Comp
-L GND #PWR0128
+L GND #PWR617
 U 1 1 5850CFB1
 P 7350 3000
-F 0 "#PWR0128" H 7220 3040 50  0001 L CNN
+F 0 "#PWR617" H 7220 3040 50  0001 L CNN
 F 1 "GND" H 7350 2900 50  0000 C CNN
 F 2 "" H 7350 3000 60  0001 C CNN
@@
 $EndComp
 $Comp
-L GND #PWR0129
+L GND #PWR621
 U 1 1 5850DCB1
 P 7800 2450
-F 0 "#PWR0129" H 7670 2490 50  0001 L CNN
+F 0 "#PWR621" H 7670 2490 50  0001 L CNN
 F 1 "GND" H 7800 2350 50  0000 C CNN
 F 2 "" H 7800 2450 60  0001 C CNN
@@
 $EndComp
 $Comp
-L GND #PWR0130
+L GND #PWR619
 U 1 1 5850DCB7
 P 7550 2450
-F 0 "#PWR0130" H 7420 2490 50  0001 L CNN
+F 0 "#PWR619" H 7420 2490 50  0001 L CNN
 F 1 "GND" H 7550 2350 50  0000 C CNN
 F 2 "" H 7550 2450 60  0001 C CNN
@@
 $EndComp
 $Comp
-L VCC #PWR0131
+L VCC #PWR618
 U 1 1 5850DD47
 P 7550 2250
-F 0 "#PWR0131" H 7550 2360 50  0001 L CNN
+F 0 "#PWR618" H 7550 2360 50  0001 L CNN
 F 1 "VCC" H 7550 2340 50  0000 C CNN
 F 2 "" H 7550 2250 60  0001 C CNN
@@
 $EndComp
 $Comp
-L VCC #PWR0132
+L VCC #PWR620
 U 1 1 5850DD8E
 P 7800 2250
-F 0 "#PWR0132" H 7800 2360 50  0001 L CNN
+F 0 "#PWR620" H 7800 2360 50  0001 L CNN
 F 1 "VCC" H 7800 2340 50  0000 C CNN
 F 2 "" H 7800 2250 60  0001 C CNN
@@
 $EndComp
 $Comp
-L VCC #PWR0133
+L VCC #PWR636
 U 1 1 5850E3EB
 P 9750 2750
-F 0 "#PWR0133" H 9750 2860 50  0001 L CNN
+F 0 "#PWR636" H 9750 2860 50  0001 L CNN
 F 1 "VCC" H 9750 2840 50  0000 C CNN
 F 2 "" H 9750 2750 60  0001 C CNN
@@
 LCD SCREEN
 $Comp
-L GND #PWR0134
+L GND #PWR630
 U 1 1 5850EBB1
 P 8350 4350
-F 0 "#PWR0134" H 8220 4390 50  0001 L CNN
+F 0 "#PWR630" H 8220 4390 50  0001 L CNN
 F 1 "GND" H 8350 4250 50  0000 C CNN
 F 2 "" H 8350 4350 60  0001 C CNN
@@
 	8350 4300 8350 4350
 $Comp
-L 3v3 #PWR0135
+L 3v3 #PWR629
 U 1 1 5850EC90
 P 8350 4150
-F 0 "#PWR0135" H 8350 4260 50  0001 L CNN
+F 0 "#PWR629" H 8350 4260 50  0001 L CNN
 F 1 "3v3" H 8350 4240 50  0000 C CNN
 F 2 "" H 8350 4150 60  0001 C CNN
@@
 	8350 4200 8450 4200
 $Comp
-L GND #PWR0136
+L GND #PWR632
 U 1 1 5850ED85
 P 9700 4300
-F 0 "#PWR0136" H 9570 4340 50  0001 L CNN
+F 0 "#PWR632" H 9570 4340 50  0001 L CNN
 F 1 "GND" H 9700 4200 50  0000 C CNN
 F 2 "" H 9700 4300 60  0001 C CNN
@@
 $EndComp
 $Comp
-L GND #PWR0137
+L GND #PWR633
 U 1 1 5850EE77
 P 9700 4500
-F 0 "#PWR0137" H 9570 4540 50  0001 L CNN
+F 0 "#PWR633" H 9570 4540 50  0001 L CNN
 F 1 "GND" H 9700 4400 50  0000 C CNN
 F 2 "" H 9700 4500 60  0001 C CNN
@@
 $EndComp
 $Comp
-L GND #PWR0138
+L GND #PWR634
 U 1 1 5850EEC1
 P 9700 4800
-F 0 "#PWR0138" H 9570 4840 50  0001 L CNN
+F 0 "#PWR634" H 9570 4840 50  0001 L CNN
 F 1 "GND" H 9700 4700 50  0000 C CNN
 F 2 "" H 9700 4800 60  0001 C CNN
@@
 $EndComp
 $Comp
-L GND #PWR0139
+L GND #PWR635
 U 1 1 5850EF0B
 P 9700 5000
-F 0 "#PWR0139" H 9570 5040 50  0001 L CNN
+F 0 "#PWR635" H 9570 5040 50  0001 L CNN
 F 1 "GND" H 9700 4900 50  0000 C CNN
 F 2 "" H 9700 5000 60  0001 C CNN
@@
 $EndComp
 $Comp
-L GND #PWR0140
+L GND #PWR627
 U 1 1 58511953
 P 8100 4200
-F 0 "#PWR0140" H 7970 4240 50  0001 L CNN
+F 0 "#PWR627" H 7970 4240 50  0001 L CNN
 F 1 "GND" H 8100 4100 50  0000 C CNN
 F 2 "" H 8100 4200 60  0001 C CNN
@@
 $EndComp
 $Comp
-L GND #PWR0141
+L GND #PWR623
 U 1 1 58511959
 P 7850 4200
-F 0 "#PWR0141" H 7720 4240 50  0001 L CNN
+F 0 "#PWR623" H 7720 4240 50  0001 L CNN
 F 1 "GND" H 7850 4100 50  0000 C CNN
 F 2 "" H 7850 4200 60  0001 C CNN
@@
 $EndComp
 $Comp
-L 3v3 #PWR0142
+L 3v3 #PWR626
 U 1 1 5851195F
 P 8100 4000
-F 0 "#PWR0142" H 8100 4110 50  0001 L CNN
+F 0 "#PWR626" H 8100 4110 50  0001 L CNN
 F 1 "3v3" H 8100 4090 50  0000 C CNN
 F 2 "" H 8100 4000 60  0001 C CNN
@@
 $EndComp
 $Comp
-L 3v3 #PWR0143
+L 3v3 #PWR622
 U 1 1 58511965
 P 7850 4000
-F 0 "#PWR0143" H 7850 4110 50  0001 L CNN
+F 0 "#PWR622" H 7850 4110 50  0001 L CNN
 F 1 "3v3" H 7850 4090 50  0000 C CNN
 F 2 "" H 7850 4000 60  0001 C CNN
@@
 $EndComp
 $Comp
-L GND #PWR0144
+L GND #PWR637
 U 1 1 58511AC2
 P 10050 4700
-F 0 "#PWR0144" H 9920 4740 50  0001 L CNN
+F 0 "#PWR637" H 9920 4740 50  0001 L CNN
 F 1 "GND" H 10050 4600 50  0000 C CNN
 F 2 "" H 10050 4700 60  0001 C CNN
@@
 $EndComp
 $Comp
-L GND #PWR0145
+L GND #PWR638
 U 1 1 58511D06
 P 10300 4700
-F 0 "#PWR0145" H 10170 4740 50  0001 L CNN
+F 0 "#PWR638" H 10170 4740 50  0001 L CNN
 F 1 "GND" H 10300 4600 50  0000 C CNN
 F 2 "" H 10300 4700 60  0001 C CNN
@@
 	10300 4500 10300 4550
 $Comp
-L GND #PWR0146
+L GND #PWR631
 U 1 1 58512287
 P 8350 4600
-F 0 "#PWR0146" H 8220 4640 50  0001 L CNN
+F 0 "#PWR631" H 8220 4640 50  0001 L CNN
 F 1 "GND" H 8350 4500 50  0000 C CNN
 F 2 "" H 8350 4600 60  0001 C CNN
@@
 	6100 4100 6100 4450
 $Comp
-L GND #PWR0147
+L GND #PWR613
 U 1 1 58512F98
 P 5500 4700
-F 0 "#PWR0147" H 5370 4740 50  0001 L CNN
+F 0 "#PWR613" H 5370 4740 50  0001 L CNN
 F 1 "GND" H 5500 4600 50  0000 C CNN
 F 2 "" H 5500 4700 60  0001 C CNN
@@
 $EndComp
 $Comp
-L GND #PWR0148
+L GND #PWR614
 U 1 1 58512FFD
 P 5700 4700
-F 0 "#PWR0148" H 5570 4740 50  0001 L CNN
+F 0 "#PWR614" H 5570 4740 50  0001 L CNN
 F 1 "GND" H 5700 4600 50  0000 C CNN
 F 2 "" H 5700 4700 60  0001 C CNN
@@
 $EndComp
 $Comp
-L GND #PWR0149
+L GND #PWR615
 U 1 1 58513062
 P 5900 4700
-F 0 "#PWR0149" H 5770 4740 50  0001 L CNN
+F 0 "#PWR615" H 5770 4740 50  0001 L CNN
 F 1 "GND" H 5900 4600 50  0000 C CNN
 F 2 "" H 5900 4700 60  0001 C CNN
@@
 $EndComp
 $Comp
-L GND #PWR0150
+L GND #PWR616
 U 1 1 585130C7
 P 6100 4700
-F 0 "#PWR0150" H 5970 4740 50  0001 L CNN
+F 0 "#PWR616" H 5970 4740 50  0001 L CNN
 F 1 "GND" H 6100 4600 50  0000 C CNN
 F 2 "" H 6100 4700 60  0001 C CNN
@@
 	5500 4650 5500 4700
 $Comp
-L 3v3 #PWR0151
+L 3v3 #PWR628
 U 1 1 58513A77
 P 8250 4500
-F 0 "#PWR0151" H 8250 4610 50  0001 L CNN
+F 0 "#PWR628" H 8250 4610 50  0001 L CNN
 F 1 "3v3" H 8250 4590 50  0000 C CNN
 F 2 "" H 8250 4500 60  0001 C CNN
@@
 Text Notes 6900 5800 0    60   ~ 0
 TOUCHSCREEN CONTROLLER
+$Comp
+L VCC #PWR608
+U 1 1 58528EF1
+P 4100 3050
+F 0 "#PWR608" H 4100 3160 50  0001 L CNN
+F 1 "VCC" H 4100 3140 50  0000 C CNN
+F 2 "" H 4100 3050 60  0001 C CNN
+F 3 "" H 4100 3050 60  0001 C CNN
+	1    4100 3050
+	1    0    0    -1
+$EndComp
 $EndSCHEMATC

Commit message: add farnell part numbers for passives
Parts:
- C601, C605, C608: Farnell (none) -> 2494230
- C602, C603, C607, C609: Farnell (none) -> 1759037
- C604, C606: Farnell (none) -> 1759011
- C610, C611: Farnell (none) -> 1759102
- R601, R602: Farnell (none) -> 9330380
- R603, R604: Farnell (none) -> 9330461
- R605: Farnell (none) -> 9330771
- R606: Farnell (none) -> 9330399
